File: eagle/proj/Dooba/dsy01.sch (EAGLE design)
At the start: 4 parts, among them U1 STM32F071LQFP100, X1 8MHz

Commit message: Added AS6C1608 2048Kb SRAM to DSY01
Parts:
- added C3: CAP, dooba:CAP
- added U2: AS6C1608TSOPII-44, dooba:AS6C1608TSOPII-44
Connections:
- new net N$10: U1.PA1, U2.DQ1
- new net N$11: U1.PA0, U2.DQ0
- new net N$12: U1.PD9, U2.A9
- new net N$13: U1.PD10, U2.A10
- new net N$14: U1.PD11, U2.A11
- new net N$15: U1.PD12, U2.A12
- new net N$16: U1.PD13, U2.A13
- new net N$17: U1.PD14, U2.A14
- new net N$18: U1.PD15, U2.A15
- new net N$19: U1.PA8, U2.A16
- new net N$20: U1.PA9, U2.A17
- new net N$21: U1.PA10, U2.A18
- new net N$22: U1.PA11, U2.A19
- new net N$23: U1.PA12, U2.A20
- new net N$24: U1.PD0, U2.A0
- new net N$25: U1.PD1, U2.A1
- new net N$26: U1.PD2, U2.A2
- new net N$27: U1.PD3, U2.A3
- new net N$28: U1.PD4, U2.A4
- new net N$29: U1.PD5, U2.A5
- new net N$3: U1.PD8, U2.A8
- new net N$30: U1.PD6, U2.A6
- new net N$31: U1.PD7, U2.A7
- new net N$4: U1.PA7, U2.DQ7
- new net N$5: U1.PA6, U2.DQ6
- new net N$6: U1.PA5, U2.DQ5
- new net N$7: U1.PA4, U2.DQ4
- new net N$8: U1.PA3, U2.DQ3
- new net N$9: U1.PA2, U2.DQ2
- net GND: now also C3.1, U2.GND_12, U2.GND_34
- net VCC: now also C3.2, U2.VCC_11, U2.VCC_33

Commit message: Further designed DSY01
Parts:
- added C10, C11: 4.7uF, dooba:CAP0805
- added C12, C13, C14, C15, C16: CAP0805, dooba:CAP0805
- added C4, C5, C7, C8: 100nF, dooba:CAP0805
- added C6: 10nF, dooba:CAP0805
- added C9: 1uF, dooba:CAP0805
- added U3: STM32F030LQFP32, dooba:STM32F030LQFP32
- C1, C2: device dooba:CAP -> dooba:CAP0805
- C3: value CAP -> 100nF; device dooba:CAP -> dooba:CAP0805
Connections:
- net GND: now also C10.1, C11.1, C12.2, C13.2, C14.2, C15.2, C16.1, C4.1, C5.2, C6.1, C7.2, C8.1, C9.1, U3.GND_16, U3.GND_32
- net VCC: now also C10.2, C11.2, C12.1, C13.1, C14.1, C15.1, C16.2, C4.2, C5.1, C6.2, C7.1, C8.2, C9.2, U3.VCCA, U3.VCC_1, U3.VCC_17

Commit message: Added Workers to DSY01 Board Added some parts to Dooba Eagle Lib (MIC550X, Pins)
Parts:
- added C17, C18, C24, C25, C31, C32, C38, C39, C45, C46, C54, C55: 27pF, dooba:CAP0805
- added C19, C21, C26, C28, C33, C35, C40, C42, C49, C51, C56: 100nF, dooba:CAP0805
- added C20, C27, C34, C41, C50: 10nF, dooba:CAP0805
- added C22, C29, C36, C43, C52: 4.7uF, dooba:CAP0805
- added C23, C30, C37, C44, C47, C48, C53: 1uF, dooba:CAP0805
- added U10: S25FLXXXSSOIC16, dooba:S25FLXXXSSOIC16
- added U4, U5, U6, U7, U9: STM32F030LQFP32, dooba:STM32F030LQFP32
- added U8: MIC550XSOT23, dooba:MIC550XSOT23
- added X2, X3, X4, X5, X6, X7: 8MHz, dooba:XTALSMD-5X32
- C12, C14: value CAP0805 -> 100nF
- C13: value CAP0805 -> 10nF
- C15: value CAP0805 -> 4.7uF
- C16: value CAP0805 -> 1uF
Connections:
- new net N$100: U1.PB4, U9.PA10
- new net N$101: U1.PC4, U9.PA11
- new net N$102: U1.PB1, U5.PA10
- new net N$103: U1.PC1, U5.PA11
- new net N$104: C38.2, U6.PF0/OSC_IN, X5.1
- new net N$105: C39.2, U6.PF1/OSC_OUT, X5.2
- new net N$106: U10.IO0/SI, U9.PB7
- new net N$107: U10.!CS, U9.PB5
- new net N$108: U10.IO1/SO, U9.PB4
- new net N$116: U1.PB2, U6.PA10
- new net N$117: U1.PC2, U6.PA11
- new net N$118: C45.2, U7.PF0/OSC_IN, X6.1
- new net N$119: C46.2, U7.PF1/OSC_OUT, X6.2
- new net N$130: U1.PB3, U7.PA10
- new net N$131: U1.PC3, U7.PA11
- new net N$32: C17.2, U3.PF0/OSC_IN, X2.1
- new net N$33: C18.2, U3.PF1/OSC_OUT, X2.2
- new net N$34: C47.2, U8.EN, U8.VIN
- new net N$43: U10.SCK, U9.PB6
- new net N$44: U1.PC0, U3.PA11
- new net N$45: C24.2, U4.PF0/OSC_IN, X3.1
- new net N$46: C25.2, U4.PF1/OSC_OUT, X3.2
- new net N$47: U4.PA0
- new net N$48: U4.PA1
- new net N$49: U4.PA2
- new net N$50: U4.PA3
- new net N$51: U4.PA4
- new net N$52: U4.PA5
- new net N$53: U4.PA6
- new net N$55: U1.PE9, U3.PA1, U5.PA1, U6.PA1, U7.PA1, U9.PA1
- new net N$56: U4.PA7
- new net N$57: U1.PB9
- new net N$58: U1.PB8
- new net N$59: U1.PB7
- new net N$60: U1.PB6
- new net N$61: U1.PB5
- new net N$63: U1.PE10, U3.PA2, U5.PA2, U6.PA2, U7.PA2, U9.PA2
- new net N$64: U1.PB10
- new net N$65: U1.PB11
- new net N$66: U1.PB12
- new net N$67: U1.PB13
- new net N$68: U1.PB14
- new net N$69: U1.PB15
- new net N$70: U4.PA9
- new net N$71: U1.PE11, U3.PA3, U5.PA3, U6.PA3, U7.PA3, U9.PA3
- new net N$72: U1.PE12, U3.PA4, U5.PA4, U6.PA4, U7.PA4, U9.PA4
- new net N$73: U1.PE13, U3.PA5, U5.PA5, U6.PA5, U7.PA5, U9.PA5
- new net N$75: U1.PC5
- new net N$76: U1.PC6
- new net N$77: U1.PC7
- new net N$78: U1.PC8
- new net N$79: U1.PC9
- new net N$80: U1.PC12
- new net N$81: U1.PC11
- new net N$82: U1.PC10
- new net N$83: U1.PC13
- new net N$84: U1.PC14/OSC32_IN
- new net N$85: U1.PC15/OSC32_OUT
- new net N$86: U1.PB0, U3.PA10
- new net N$87: U4.PA8
- new net N$88: U4.PA10
- new net N$89: U4.PA11
- new net N$90: C31.2, U5.PF0/OSC_IN, X4.1
- new net N$91: C32.2, U5.PF1/OSC_OUT, X4.2
- new net N$93: U1.PE14, U3.PA6, U5.PA6, U6.PA6, U7.PA6, U9.PA6
- new net N$94: U1.PE15, U3.PA7, U5.PA7, U6.PA7, U7.PA7, U9.PA7
- new net N$95: U1.PE1, U3.PA9, U5.PA9, U6.PA9, U7.PA9, U9.PA9
- new net N$96: U1.PE0, U3.PA8, U5.PA8, U6.PA8, U7.PA8, U9.PA8
- new net N$97: U1.PE8, U3.PA0, U5.PA0, U6.PA0, U7.PA0, U9.PA0
- new net N$98: C54.2, U9.PF0/OSC_IN, X7.1
- new net N$99: C55.2, U9.PF1/OSC_OUT, X7.2
- net GND: now also C17.1, C18.1, C19.2, C20.2, C21.2, C22.2, C23.1, C24.1, C25.1, C26.2, C27.2, C28.2, C29.2, C30.1, C31.1, C32.1, C33.2, C34.2, C35.2, C36.2, C37.1, C38.1, C39.1, C40.2, C41.2, C42.2, C43.2, C44.1, C45.1, C46.1, C47.1, C48.1, C49.2, C50.2, C51.2, C52.2, C53.1, C54.1, C55.1, C56.1, U10.GND, U4.GND_16, U4.GND_32, U5.GND_16, U5.GND_32, U6.GND_16, U6.GND_32, U7.GND_16, U7.GND_32, U8.GND, U9.GND_16, U9.GND_32
- net VCC: now also C19.1, C20.1, C21.1, C22.1, C23.2, C26.1, C27.1, C28.1, C29.1, C30.2, C33.1, C34.1, C35.1, C36.1, C37.2, C40.1, C41.1, C42.1, C43.1, C44.2, C48.2, C49.1, C50.1, C51.1, C52.1, C53.2, C56.2, U10.RFU/!RST, U10.VCC, U10.VIO/RFU, U4.VCCA, U4.VCC_1, U4.VCC_17, U5.VCCA, U5.VCC_1, U5.VCC_17, U6.VCCA, U6.VCC_1, U6.VCC_17, U7.VCCA, U7.VCC_1, U7.VCC_17, U8.VOUT, U9.VCCA, U9.VCC_1, U9.VCC_17
Other:
- note added: "NOT => PA10 RDY => PA11"
- note added: "NOT => PA10 RDY => PA11 CKI => PA8 CKO => PA9 DIO[0-7] => PA[0-7]"
- note added: "NOT[0-15] => PB RDY[0-15] => PC CKI => PE0 CKO => PE1 DIO[0-7] => PE[8-15]"
- moved on the sheet: C12, C13, C14, C15, C16, U3

Commit message: Added more Pin headers to Dooba Eagle Lib Added RST signal and extension header to DSY01
Parts:
- added P1: DIO, dooba:PIN_8
- added P2: CKI-CKO, dooba:PIN_2
- added P3: NOT, dooba:PIN_11
- added P4: RDY, dooba:PIN_11
- added P5: PWR(VIN-GND-RST), dooba:PIN_3
Connections:
- new net N$35: P5.3, U1.!RST, U3.!RST, U5.!RST, U6.!RST, U7.!RST, U9.!RST
- new net N$36: U1.PE2, U2.!OE
- new net N$37: U1.PE3, U2.!WE
- new net N$38: U1.PE4, U2.CE2
- new net N$39: U1.PE5, U2.!CE
- net GND: now also P5.2
- net N$34: now also P5.1
- net N$55: now also P1.2
- net N$57: now also P3.5
- net N$58: now also P3.4
- net N$59: now also P3.3
- net N$60: now also P3.2
- net N$61: now also P3.1
- net N$63: now also P1.3
- net N$64: now also P3.6
- net N$65: now also P3.7
- net N$66: now also P3.8
- net N$67: now also P3.9
- net N$68: now also P3.10
- net N$69: now also P3.11
- net N$71: now also P1.4
- net N$72: now also P1.5
- net N$73: now also P1.6
- net N$75: now also P4.1
- net N$76: now also P4.2
- net N$77: now also P4.3
- net N$78: now also P4.4
- net N$79: now also P4.5
- net N$80: now also P4.8
- net N$81: now also P4.7
- net N$82: now also P4.6
- net N$83: now also P4.9
- net N$84: now also P4.10
- net N$85: now also P4.11
- net N$93: now also P1.7
- net N$94: now also P1.8
- net N$95: now also P2.2
- net N$96: now also P2.1
- net N$97: now also P1.1

Commit message: Added CAM and DRU files for Eagle Further routed DSY01 board
Parts:
- removed C19, C21: 100nF, dooba:CAP0805
- removed C20: 10nF, dooba:CAP0805
- removed C22: 4.7uF, dooba:CAP0805
- removed C23: 1uF, dooba:CAP0805
- removed C24, C25: 27pF, dooba:CAP0805
- removed U4: STM32F030LQFP32, dooba:STM32F030LQFP32
- removed X3: 8MHz, dooba:XTALSMD-5X32
- added P10, P11, P6, P7, P8, P9: SWD_CORE(SWCLK-SWDIO-GND), dooba:PIN_3
Connections:
- removed net N$56: U4.PA7
- removed net N$70: U4.PA9
- removed net N$87: U4.PA8
- removed net N$88: U4.PA10
- removed net N$89: U4.PA11
- new net N$40: P6.1, U1.PA14/SWCLK
- new net N$41: P6.2, U1.PA13/SWDIO
- new net N$42: P7.2, U3.PA13/SWDIO
- net GND: now also P10.3, P11.3, P6.3, P7.3, P8.3, P9.3, U1.BOOT0, U3.BOOT0, U5.BOOT0, U6.BOOT0, U7.BOOT0, U9.BOOT0; no longer C19.2, C20.2, C21.2, C22.2, C23.1, C24.1, C25.1, U4.GND_16, U4.GND_32
- net N$45: now also P10.1, U7.PA14/SWCLK; no longer C24.2, U4.PF0/OSC_IN, X3.1
- net N$46: now also P8.2, U5.PA13/SWDIO; no longer C25.2, U4.PF1/OSC_OUT, X3.2
- net N$47: now also P9.1, U6.PA14/SWCLK; no longer U4.PA0
- net N$48: now also P9.2, U6.PA13/SWDIO; no longer U4.PA1
- net N$49: now also P8.1, U5.PA14/SWCLK; no longer U4.PA2
- net N$50: now also P10.2, U7.PA13/SWDIO; no longer U4.PA3
- net N$51: now also P7.1, U3.PA14/SWCLK; no longer U4.PA4
- net N$52: now also P11.2, U9.PA13/SWDIO; no longer U4.PA5
- net N$53: now also P11.1, U9.PA14/SWCLK; no longer U4.PA6
- net VCC: no longer C19.1, C20.1, C21.1, C22.1, C23.2, U4.VCCA, U4.VCC_1, U4.VCC_17
Other:
- note removed: "NOT => PA10 RDY => PA11"

Commit message: Further designed DSY01 Board & Schematic
Parts:
- P10, P11, P6, P7, P8, P9: device dooba:PIN_3 -> dooba:PIN_2
Connections:
- net GND: now also U1.PA15, U1.PE6, U1.PE7, U1.PF10, U1.PF2, U1.PF3, U1.PF6, U1.PF9, U3.PA12, U3.PA15, U3.PB0, U3.PB1, U3.PB3, U3.PB4, U3.PB5, U3.PB6, U3.PB7, U5.PA12, U5.PA15, U5.PB0, U5.PB1, U5.PB3, U5.PB4, U5.PB5, U5.PB6, U5.PB7, U6.PA12, U6.PA15, U6.PB0, U6.PB1, U6.PB3, U6.PB4, U6.PB5, U6.PB6, U6.PB7, U7.PA12, U7.PA15, U7.PB0, U7.PB1, U7.PB3, U7.PB4, U7.PB5, U7.PB6, U7.PB7, U9.PA12, U9.PA15, U9.PB0, U9.PB1, U9.PB3; no longer P10.3, P11.3, P6.3, P7.3, P8.3, P9.3

Commit message: Finished routing DSY01 Added LEDs on DSY01
Parts:
- added D1, D2, D3, D4, D5, D6: LED0805, dooba:LED0805
- added R1, R2, R3, R4, R5, R6: 330, dooba:RES0805
Connections:
- new net N$109: R5.2, U9.PA15
- new net N$110: D6.1, R6.1
- new net N$111: R6.2, U1.PF9
- new net N$54: D1.1, R1.1
- new net N$56: R1.2, U3.PA15
- new net N$62: D2.1, R2.1
- new net N$70: R2.2, U5.PA15
- new net N$74: D3.1, R3.1
- new net N$87: R3.2, U6.PA15
- new net N$88: D4.1, R4.1
- new net N$89: R4.2, U7.PA15
- new net N$92: D5.1, R5.1
- net GND: now also D1.2, D2.2, D3.2, D4.2, D5.2, D6.2; no longer U1.PF9, U3.PA15, U5.PA15, U6.PA15, U7.PA15, U9.PA15

Commit message: Added more decorations to DSY01
Parts:
- added D7: LED0805, dooba:LED0805
- added R7: 330, dooba:RES0805
- U8: value MIC550XSOT23 -> AP2112SOT23; device dooba:MIC550XSOT23 -> dooba:AP2112SOT23
Connections:
- new net N$112: D7.1, R7.1
- net GND: now also D7.2
- net VCC: now also R7.2
Changed lines of the file:
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@@
 <part name="C46" library="dooba" deviceset="CAP" device="0805" value="27pF"/>
 <part name="GND37" library="supply1" deviceset="GND" device=""/>
-<part name="U8" library="dooba" deviceset="MIC550X" device="SOT23"/>
+<part name="U8" library="dooba" deviceset="AP2112" device="SOT23"/>
 <part name="C47" library="dooba" deviceset="CAP" device="0805" value="1uF"/>
 <part name="C48" library="dooba" deviceset="CAP" device="0805" value="1uF"/>
@@
 <part name="R6" library="dooba" deviceset="RES" device="0805" value="330"/>
 <part name="GND49" library="supply1" deviceset="GND" device=""/>
+<part name="D7" library="dooba" deviceset="LED" device="0805"/>
+<part name="R7" library="dooba" deviceset="RES" device="0805" value="330"/>
+<part name="GND61" library="supply1" deviceset="GND" device=""/>
 </parts>
 <sheets>
@@
 <instance part="R6" gate="R1" x="381" y="416.56"/>
 <instance part="GND49" gate="1" x="396.24" y="424.18" rot="R90"/>
+<instance part="D7" gate="D1" x="1534.16" y="1120.14" rot="R90"/>
+<instance part="R7" gate="R1" x="1541.78" y="1120.14" rot="R90"/>
+<instance part="GND61" gate="1" x="1534.16" y="1135.38" rot="R180"/>
 </instances>
 <busses>
@@
 <wire x1="429.26" y1="401.32" x2="431.8" y2="401.32" width="0.1524" layer="91"/>
 </segment>
+<segment>
+<pinref part="D7" gate="D1" pin="2"/>
+<pinref part="GND61" gate="1" pin="GND"/>
+<wire x1="1534.16" y1="1130.3" x2="1534.16" y2="1132.84" width="0.1524" layer="91"/>
+</segment>
 </net>
 <net name="VCC" class="0">
@@
 <wire x1="1549.4" y1="1130.3" x2="1551.94" y2="1130.3" width="0.1524" layer="91"/>
 <junction x="1549.4" y="1130.3"/>
+<pinref part="R7" gate="R1" pin="2"/>
+<wire x1="1549.4" y1="1130.3" x2="1541.78" y2="1130.3" width="0.1524" layer="91"/>
 </segment>
 <segment>
@@
 </segment>
 </net>
+<net name="N$112" class="0">
+<segment>
+<pinref part="R7" gate="R1" pin="1"/>
+<pinref part="D7" gate="D1" pin="1"/>
+<wire x1="1541.78" y1="1109.98" x2="1534.16" y2="1109.98" width="0.1524" layer="91"/>
+</segment>
+</net>
