File: eagle/proj/Dooba/dsy01.sch (EAGLE design)
At the start: 89 parts, among them P1 DIO, P10 SWD_CORE(SWCLK-SWDIO-GND), P11 SWD_CORE(SWCLK-SWDIO-GND), P2 CKI-CKO, P3 NOT, P4 RDY, P5 PWR(VIN-GND-RST), P6 SWD_CORE(SWCLK-SWDIO-GND), P7 SWD_CORE(SWCLK-SWDIO-GND), P8 SWD_CORE(SWCLK-SWDIO-GND)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

Commit message: Finished decorating (?) DSY01
Parts:
- added P12: SWD(GND-RST), dooba:PIN_2
Connections:
- net GND: now also P12.1
- net N$35: now also P12.2
Changed lines of the file:
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@@
 <part name="R7" library="dooba" deviceset="RES" device="0805" value="330"/>
 <part name="GND61" library="supply1" deviceset="GND" device=""/>
+<part name="P12" library="dooba" deviceset="PIN_2" device="" value="SWD(GND-RST)"/>
+<part name="GND62" library="supply1" deviceset="GND" device=""/>
 </parts>
 <sheets>
@@
 <instance part="R7" gate="R1" x="1541.78" y="1120.14" rot="R90"/>
 <instance part="GND61" gate="1" x="1534.16" y="1135.38" rot="R180"/>
+<instance part="P12" gate="P1" x="1615.44" y="1112.52"/>
+<instance part="GND62" gate="1" x="1602.74" y="1112.52" rot="R270"/>
 </instances>
 <busses>
@@
 <pinref part="GND61" gate="1" pin="GND"/>
 <wire x1="1534.16" y1="1130.3" x2="1534.16" y2="1132.84" width="0.1524" layer="91"/>
+</segment>
+<segment>
+<pinref part="GND62" gate="1" pin="GND"/>
+<pinref part="P12" gate="P1" pin="1"/>
+<wire x1="1605.28" y1="1112.52" x2="1607.82" y2="1112.52" width="0.1524" layer="91"/>
 </segment>
 </net>
@@
 <pinref part="P5" gate="P1" pin="3"/>
 <wire x1="1607.82" y1="1125.22" x2="1602.74" y2="1125.22" width="0.1524" layer="91"/>
-<wire x1="1602.74" y1="1125.22" x2="1579.88" y2="1102.36" width="0.1524" layer="91"/>
+<wire x1="1602.74" y1="1125.22" x2="1587.5" y2="1109.98" width="0.1524" layer="91"/>
+<wire x1="1587.5" y1="1109.98" x2="1579.88" y2="1102.36" width="0.1524" layer="91"/>
 <wire x1="1579.88" y1="1102.36" x2="426.72" y2="1102.36" width="0.1524" layer="91"/>
 <wire x1="426.72" y1="1102.36" x2="218.44" y2="894.08" width="0.1524" layer="91"/>
@@
 <wire x1="1239.52" y1="784.86" x2="960.12" y2="784.86" width="0.1524" layer="91"/>
 <junction x="960.12" y="784.86"/>
-</segment>
-</net>
+<pinref part="P12" gate="P1" pin="2"/>
+<wire x1="1607.82" y1="1109.98" x2="1587.5" y2="1109.98" width="0.1524" layer="91"/>
+<junction x="1587.5" y="1109.98"/>
+</segment>
+</net>
