File: eagle/proj/Dooba/dsy01.brd (EAGLE design)
At the start: 66.2 x 70.1 mm, 87 parts, among them P1 DIO, P10 SWD_CORE(SWCLK-SWDIO-GND), P11 SWD_CORE(SWCLK-SWDIO-GND), P2 CKI-CKO, P3 NOT, P4 RDY, P5 PWR(VIN-GND-RST), P6 SWD_CORE(SWCLK-SWDIO-GND), P7 SWD_CORE(SWCLK-SWDIO-GND), P8 SWD_CORE(SWCLK-SWDIO-GND)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

Commit message: Added more decorations to DSY01
Parts:
- added D7: LED0805, dooba:0805
- added R7: 330, dooba:0805
- U8: value MIC550XSOT23 -> AP2112SOT23
Connections:
- new net N$112: D7.1, R7.1
- net GND: now also D7.2
- net VCC: now also R7.2
Routing:
- net N$112: track 0.00 -> 1.38 mm
- net VCC: track 569.5 -> 570.5 mm
Other:
- board text added: "---------> 330R"
- board text added: "-----> LED"
- board text added: "8Mhz"
- board text added: "AS6C1608"
- board text added: "S25FL256S"
- board text added: "STM32F030"
- board text added: "STM32F071"
- board text added: "VIN: 4-6V 600mA Core: 2Mb RAM SFSU: 32Mb Flash Workers: 4 Holes: 2.2mm"

Commit message: Finished decorating (?) DSY01
Parts:
- added P12: SWD(GND-RST), dooba:PIN_2
Connections:
- net GND: now also P12.1
- net N$35: now also P12.2
Routing:
- net N$35: track 149.6 -> 154.4 mm
- net GND: vias 245 -> 243
Other:
- board text added: "0"
- board text added: "15"
- board text added: "5"
- board text added: "7"
- board text added: "AP2112"
- board text added: "CK"
- board text added: "CKI"
- board text added: "CKO"
- board text added: "Core SWD"
- board text added: "DIO"
- board text added: "DSY01 Dooba System Board [ 4x WKR / 2Mb Core / 64Mb SFSU ] Power Supply: 4-6V 600mA Nov 2016 <eresse@eresse.net>"
- board text added: "GND"
- board text added: "IO"
- board text added: "NOT"
- board text added: "RDY"
- board text added: "RST"
- board text added: "SFSU SWD"
- board text added: "VIN"
- board text added: "Worker SWD"
