File: eagle/proj/Dooba/ionode_sunb.sch (EAGLE design)
At the start: 42 parts, among them J1 USB-BAMPHENOL-MICRO, U1 TPS61200S-PVSON-N10, U2 MAX1811SO8, U3 FT232RQFN32, U4 MCP4018SC70, U5 DIPSWITCH_2DIP, U6 AP7335SOT23-5

Commit message: Started shiva mp3 player board
Parts:
- added P1: ICSP(RST-MOSI-MISO-SCK), dooba:PIN_4
- added R14, R15, R16, R17: 10k, dooba:RES0805
- added SW1, SW2, SW3, SW4: TACTSWCK_PTS_830, dooba:TACTSWCK_PTS_830
- R11: value TRIMPOTBOURNS-3306F -> LCD_CONTRAST
- U5: value DIPSWITCH_2DIP -> UART_DCNT
Connections:
- new net N$21: IO[8-15].5, R14.2, SW1.4
- new net N$22: IO[8-15].4, R15.2, SW2.4
- new net N$23: IO[8-15].3, R16.2, SW3.4
- new net N$24: IO[0-7].8, R17.2, SW4.4
- new net N$25: ISP(SCK-MISO).1, P1.4
- new net N$26: ISP(MOSI-RST).2, P1.1
- net GND: now also R14.1, R15.1, R16.1, R17.1, U1.PAD0, U1.PAD1, U1.PAD2, U1.PAD3
- net LCD_BACKLIGHT_SCL: now also R12.2
- net LCD_BACKLIGHT_SDA: no longer R12.2
- net N$1: now also P1.2
- net N$16: now also P1.3
- net VCC: now also SW1.1, SW2.1, SW3.1, SW4.1
Other:
- moved on the sheet: C2, R12, R13, R3, R4
