File: eagle/proj/Dooba/shiva.sch (EAGLE design)
At the start: 116 parts, among them J1 DM3D-SFDM, J2 USB-BAMPHENOL-MICRO, J3 SJ1-3523N, J4 ADAFRUIT_OLED_13, SW1 LEFT, SW2 UP, SW3 CENTER, SW4 DOWN, SW5 RIGHT, SW6 VOL_UP, SW7 VOL_DN, U1 STM32F030X-LQFP48LQFP48, U10 CS4334, U11 LM4811PDSO-10, U12 5.0V, U13 MCP23008QFN, U2 TPS61200S-PVSON-N10, U3 MAX1811SO8, U4 FT232RQFN32, U5 SN74LVC1G125SOT23-5, U6 SN74LVC1G125SOT23-5, U7 3.3V, U8 3.3V, U9 STA013LQFP44, X1 16MHz, X2 14.7456MHz

Commit message: Added BOM Tools Completed Shiva MP3 Player Board
Parts:
- removed C12, C4: 100nF, dooba:CAP0805
- removed C13, C3: 4.7uF, dooba:CAP0805
- removed C14: 22uF, dooba:CAP_POLARIZEDSMD_RADIAL_43
- removed R23, R24, R25, R26, R27, R28, R29: 10k, dooba:RES0805
- added P1: PB[2-3-4], dooba:PIN_3
- added P2: PB5-PB6/SCL-PB7/SDA, dooba:PIN_3
- added P3: PB[8-9-10], dooba:PIN_3
- added P4: PF6-PF7-PA8, dooba:PIN_3
- added P5: PA[11-12-15], dooba:PIN_3
- added P6: PA13/SWDIO-PA14/SWCLK-RST, dooba:PIN_3
- added P7: 5.5V-USBVCC-GND, dooba:PIN_3
- added P8: 5.5V-BATTVCC-GND, dooba:PIN_3
- added P9: AOUT_L-GND-AOUT_R, dooba:PIN_3
- added S1: SWITCH_SPSTGF-1123-0025, dooba:SWITCH_SPSTGF-1123-0025
- C2: value 100nF -> 10uF
- C39: value CAP_POLARIZEDSMD_RADIAL_43 -> 10uF
- C40, C41: value CAP_POLARIZEDSMD_RADIAL_43 -> 3.3uF
- C42: value CAP0805 -> 100nF
- C43, C44: value CAP0805 -> 3.3nF
- C47, C50, C51, C52: value CAP_POLARIZEDSMD_RADIAL_43 -> 1uF
- C48, C49: value CAP_POLARIZEDSMD_RADIAL_43 -> 100uF; device dooba:CAP_POLARIZEDSMD_RADIAL_43 -> dooba:CAP_POLARIZEDSMD_RADIAL_66
- R16, R17: value RES0805 -> 560R
- R18, R19: value RES0805 -> 270k
- R22: value RES0805 -> 100k
- SW1: value LEFT -> VD
- SW2: value UP -> D
- SW3: value CENTER -> R
- SW4: value DOWN -> VU
- SW5: value RIGHT -> C
- SW6: value VOL_UP -> U
- SW7: value VOL_DN -> L
Connections:
- new net BATT_PWR: BATT(VCC-GND).1, C2.1, R6.1, R7.1, S1.1, U3.BATT, U3.EN
- new net N$47: P3.3, U1.PB10
- new net N$48: P3.2, U1.PB9
- new net N$49: P3.1, U1.PB8
- new net N$50: P2.1, U1.PB5
- new net N$51: P1.3, U1.PB4
- new net N$52: P1.2, U1.PB3
- new net N$53: P1.1, U1.PB2
- new net N$54: P4.3, U1.PA8
- new net N$55: P4.1, U1.PF6
- new net N$56: P4.2, U1.PF7
- new net N$57: P5.1, U1.PA11
- new net N$58: P5.2, U1.PA12
- new net N$59: P5.3, U1.PA15
- new net N$60: P6.1, U1.PA13/SWDIO
- new net N$61: P6.2, U1.PA14/SWCLK
- net 3.3V-CORE: now also R20.1, R21.1; no longer C12.1, C13.1, C2.1, C3.1, C4.1, R23.1, R24.1, R25.1, R26.1, R27.1, R28.1, R29.1
- net 3.3V-MICROSD: no longer C14.2
- net 5.5V: now also P7.1, P8.1
- net AOUT_L: now also P9.1
- net AOUT_R: now also P9.3
- net BATTVCC: now also P8.2, S1.2; no longer BATT(VCC-GND).1, R6.1, R7.1, U3.BATT, U3.EN
- net GND: now also P7.3, P8.3, P9.2; no longer C12.2, C13.2, C14.1, C3.2, C4.2, R20.1, R21.1
- net I2C_SCL: now also P2.2
- net I2C_SDA: now also P2.3
- net N$1: now also P6.3
- net N$33: no longer R23.2
- net N$35: no longer R24.2
- net N$36: no longer R25.2
- net N$37: no longer R26.2
- net N$38: no longer R27.2
- net N$41: no longer R28.2
- net N$42: no longer R29.2
- net USBVCC: now also P7.2
Other:
- note added: "Audio Blocks - CS4334 D/A Converter - LM4811 Headphone Amp"
- note added: "Core Logic Blocks Includes - STM32F030 Microcontroller - STA013 MP3 Decoder"
- note added: "MicroSD Block Includes uSD Card reader"
- note added: "UI Blocks - 128x64 Monochrome OLED - MCP23008 I/O Expander + 7 Buttons"
- note added: "USB & Power Blocks Include USB LiPo Charger Provides USB UART"
- moved on the sheet: BATT(VCC-GND), C1, C10, C11, C2, C27, C5, C6, C7, C8, C9, D4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

Commit message: Started designing Shiva mp3 player (new version)
Parts:
- removed BATT(VCC-GND): PIN_2, dooba:PIN_2
- removed C10, C30, C31, C9: 27pF, dooba:CAP0805
- removed C11, C16, C18, C19, C23, C24, C27, C32, C33, C34, C35, C36, C42: 100nF, dooba:CAP0805
- removed C15, C8: 4.7uF, dooba:CAP0805
- removed C17: 22uF, dooba:CAP1206
- removed C20: 10uF, dooba:CAP0805
- removed C21, C39: 10uF, dooba:CAP_POLARIZEDSMD_RADIAL_43
- removed C22: 4.7uF, dooba:CAP_POLARIZEDSMD_RADIAL_43
- removed C25, C26, C28, C29, C45, C46, C7: 1uF, dooba:CAP0805
- removed C37: 470pF, dooba:CAP0805
- removed C38: 4.7nF, dooba:CAP0805
- removed C40, C41: 3.3uF, dooba:CAP_POLARIZEDSMD_RADIAL_43
- removed C43, C44: 3.3nF, dooba:CAP0805
- removed C47, C50, C51, C52: 1uF, dooba:CAP_POLARIZEDSMD_RADIAL_43
- removed C48, C49: 100uF, dooba:CAP_POLARIZEDSMD_RADIAL_66
- removed C6: 10nF, dooba:CAP0805
- removed D1: CHARGE, dooba:LED0805
- removed D2: TX, dooba:LED0805
- removed D3: RX, dooba:LED0805
- removed D4: MicroSD, dooba:LED0805
- removed D5: Activity, dooba:LED0805
- removed J3: SJ1-3523N, dooba:SJ1-3523N
- removed J4: ADAFRUIT_OLED_13, dooba:ADAFRUIT_OLED_13
- removed L1: 4.7uH, dooba:INDSMD-3232
- removed P1: PB[2-3-4], dooba:PIN_3
- removed P2: PB5-PB6/SCL-PB7/SDA, dooba:PIN_3
- removed P3: PB[8-9-10], dooba:PIN_3
- removed P4: PF6-PF7-PA8, dooba:PIN_3
- removed P5: PA[11-12-15], dooba:PIN_3
- removed P6: PA13/SWDIO-PA14/SWCLK-RST, dooba:PIN_3
- removed P7: 5.5V-USBVCC-GND, dooba:PIN_3
- removed P8: 5.5V-BATTVCC-GND, dooba:PIN_3
- removed P9: AOUT_L-GND-AOUT_R, dooba:PIN_3
- removed R10, R15, R30, R31, R8, R9: 1k, dooba:RES0805
- removed R11: 1M, dooba:RES0805
- removed R12, R13: 4.7R, dooba:RES0805
- removed R14, R20, R21, R6, R7: 10k, dooba:RES0805
- removed R16, R17: 560R, dooba:RES0805
- removed R18, R19: 270k, dooba:RES0805
- removed R22: 100k, dooba:RES0805
- removed R3, R5: 200k, dooba:RES0805
- removed R4: 2M, dooba:RES0805
- removed U10: CS4334, dooba:CS4334
- removed U11: LM4811PDSO-10, dooba:LM4811PDSO-10
- removed U12: 5.0V, dooba:LP3985SOT23-5
- removed U13: MCP23008QFN, dooba:MCP23008QFN
- removed U5, U6: SN74LVC1G125SOT23-5, dooba:SN74LVC1G125SOT23-5
- removed U7, U8: 3.3V, dooba:LP3985SOT23-5
- removed U9: STA013LQFP44, dooba:STA013LQFP44
- removed X1: 16MHz, dooba:XTAL_GNDSMD_3225
- removed X2: 14.7456MHz, dooba:XTAL_GNDSMD_3225
- added C3: 10uF, dooba:CAP0805
- added C4: 100nF, dooba:CAP0805
- added N1: DOOBA_IONODE, dooba:DOOBA_IONODE
- C1: value 100nF -> 1uF
- C2: value 10uF -> 1uF
- J2: value USB-BAMPHENOL-MICRO -> ADAFRUIT_OLED_13; device dooba:USB-BAMPHENOL-MICRO -> dooba:ADAFRUIT_OLED_13
- R2: value 2M -> 10k
- S1: value SWITCH_SPSTGF-1123-0025 -> PWR; device dooba:SWITCH_SPSTGF-1123-0025 -> dooba:SWITCH_SPDT
- SW1: value VD -> TACTSWB3SL-10XXP; device dooba:TACTSWCK_PTS_830 -> dooba:TACTSWB3SL-10XXP
- SW2: value D -> TACTSWB3SL-10XXP; device dooba:TACTSWCK_PTS_830 -> dooba:TACTSWB3SL-10XXP
- SW3: value R -> TACTSWB3SL-10XXP; device dooba:TACTSWCK_PTS_830 -> dooba:TACTSWB3SL-10XXP
- SW4: value VU -> TACTSWB3SL-10XXP; device dooba:TACTSWCK_PTS_830 -> dooba:TACTSWB3SL-10XXP
- SW5: value C -> TACTSWB3SL-10XXP; device dooba:TACTSWCK_PTS_830 -> dooba:TACTSWB3SL-10XXP
- SW6: value U -> TACTSWB3SL-10XXP; device dooba:TACTSWCK_PTS_830 -> dooba:TACTSWB3SL-10XXP
- SW7: value L -> TACTSWB3SL-10XXP; device dooba:TACTSWCK_PTS_830 -> dooba:TACTSWB3SL-10XXP
- U1: value STM32F030X-LQFP48LQFP48 -> MCP23008QFN; device dooba:STM32F030X-LQFP48LQFP48 -> dooba:MCP23008QFN
- U2: value TPS61200S-PVSON-N10 -> DOOBA_AECHO_NOAOUT; device dooba:TPS61200S-PVSON-N10 -> dooba:DOOBA_AECHO_NOAOUT
- U3: value MAX1811SO8 -> DOOBA_NOMAD; device dooba:MAX1811SO8 -> dooba:DOOBA_NOMAD
- U4: value FT232RQFN32 -> 3.3V; device dooba:FT232RQFN32 -> dooba:LP3985SOT23-5
Connections:
- removed net !MICROSD_CS: J1.DAT3/CS, U1.PB15
- removed net !STA013_RST: R14.1, U1.PA3, U9.!RESET
- removed net 3.3V-CORE: C1.1, C11.1, C26.1, C32.2, C33.2, C34.2, C35.2, C5.1, C6.2, C7.2, C8.1, R13.1, R14.2, R20.1, R21.1, U1.VCC@1, U1.VCC@24, U1.VCC@48, U1.VCCA, U13.!RST, U13.A2, U13.VCC, U5.!OE, U5.VCC, U7.VOUT, U9.!SRC_INT, U9.!TESTEN, U9.BIT_EN, U9.VDD_1, U9.VDD_2, U9.VDD_3, U9.VDD_4
- removed net 3.3V-MICROSD: C15.2, C16.2, C29.1, J1.VCC, R1.1, U8.VOUT
- removed net 5.0V-AUDIO: C39.2, C42.1, C46.1, C47.2, R22.2, U10.VA, U11.VCC, U12.VOUT
- removed net AMP_SHUTDOWN: R22.1, U1.PA2, U11.SHUTDOWN
- removed net AMP_VOL_CLK: U1.PA1, U11.CLOCK
- removed net AMP_VOL_UPDN: U1.PA0, U11.UP/DN
- removed net AOUT_L: C43.1, C51.1, P9.1, R17.2
- removed net AOUT_R: C44.2, C52.1, P9.3, R16.2
- removed net BATTVCC: C19.2, C20.2, L1.2, P8.2, R2.2, S1.2, U2.EN, U2.PS, U2.VIN
- removed net BATT_PWR: BATT(VCC-GND).1, C2.1, R6.1, R7.1, S1.1, U3.BATT, U3.EN
- removed net FT232R_RX: U4.RXD, U6.Y
- removed net FT232R_TX: U4.TXD, U5.A
- removed net MICROSD_DET: J1.DET_A, R1.2, U1.PB11
- removed net N$10: C40.2, R18.1, U10.AOUTL
- removed net N$12: C41.2, R19.2, U10.AOUTR
- removed net N$13: C19.1, R2.1, R3.1, U2.UVLO
- removed net N$14: R4.1, R5.1, U2.FB
- removed net N$15: C18.2, U2.VAUX
- removed net N$16: L1.1, U2.L
- removed net N$17: D1.2, U3.!CHG
- removed net N$18: D1.1, R8.2
- removed net N$19: R7.2, U3.SELV
- removed net N$20: R6.2, U3.SELI
- removed net N$21: C24.2, U4.3V3OUT
- removed net N$22: D2.2, U4.CBUS0
- removed net N$23: D3.2, U4.CBUS1
- removed net N$24: D2.1, R9.2
- removed net N$25: D3.1, R10.2
- removed net N$26: J2.D-, U4.USBDM
- removed net N$27: J2.D+, U4.USBDP
- removed net N$28: C41.1, R16.1
- removed net N$29: C40.1, R17.1
- removed net N$30: C48.2, U11.VOUT1
- removed net N$31: C49.2, U11.VOUT2
- removed net N$32: C50.2, U11.BYPASS
- removed net N$33: SW1.1, U13.GP0
- removed net N$34: C49.1, J3.RING
- removed net N$35: SW2.1, U13.GP1
- removed net N$36: SW3.1, U13.GP2
- removed net N$37: SW4.1, U13.GP3
- removed net N$38: SW5.1, U13.GP4
- removed net N$39: C51.2, U11.VIN1
- removed net N$40: C52.2, U11.VIN2
- removed net N$41: SW6.1, U13.GP5
- removed net N$42: SW7.1, U13.GP6
- removed net N$43: D4.1, R30.2
- removed net N$44: D5.1, R31.2
- removed net N$45: R30.1, U1.PB1
- removed net N$46: R31.1, U1.PB0
- removed net N$47: P3.3, U1.PB10
- removed net N$48: P3.2, U1.PB9
- removed net N$49: P3.1, U1.PB8
- removed net N$50: P2.1, U1.PB5
- removed net N$51: P1.3, U1.PB4
- removed net N$52: P1.2, U1.PB3
- removed net N$53: P1.1, U1.PB2
- removed net N$54: P4.3, U1.PA8
- removed net N$55: P4.1, U1.PF6
- removed net N$56: P4.2, U1.PF7
- removed net N$57: P5.1, U1.PA11
- removed net N$58: P5.2, U1.PA12
- removed net N$59: P5.3, U1.PA15
- removed net N$60: P6.1, U1.PA13/SWDIO
- removed net N$61: P6.2, U1.PA14/SWCLK
- removed net N$8: C48.1, J3.TIP
- removed net N$9: C38.2, R15.2
- removed net STA013_DREQ: U1.PA6, U9.OUT_CLK/DATA_REC
- removed net STA013_LRCKT: U10.LRCK, U9.LRCKT
- removed net STA013_OCLK: U10.MCLK, U9.OCLK
- removed net STA013_SCKR: U1.PA5, U9.SCKR
- removed net STA013_SCKT: U10.DEM/SCLK, U9.SCKT
- removed net STA013_SDI: U1.PA7, U9.SDI
- removed net STA013_SDO: U10.SDATA, U9.SDO
- removed net STM32F0_RX: U1.PA10/USART1_RX, U5.Y
- removed net STM32F0_TX: U1.PA9/USART1_TX, U6.A
- removed net USBVCC: C21.2, C22.2, C23.2, J2.VCC, P7.2, R10.1, R8.1, R9.1, U3.IN, U4.!RESET, U4.VCC, U4.VCCIO, U6.!OE, U6.VCC
- new net 3.3V: C2.2, C3.1, C4.1, C5.1, J1.VCC, R1.2, R2.2, U1.!RST, U1.A2, U1.VCC, U4.VOUT
- new net AMP_CLK: N1.PD6, U2.AMP_CLK
- new net AMP_SHDN: N1.PD7, U2.AMP_SHDN
- new net AMP_VUPDN: N1.PD5, U2.AMP_VUPDN
- new net MICROSD_CS: J1.DAT3/CS, N1.PB3
- new net MP3_DREQ: N1.PC6, U2.MP3_DREQ
- new net MP3_RST: N1.PC7, U2.MP3_RST
- new net MP3_SCKR: N1.PC4, U2.MP3_SCKR
- new net MP3_SDI: N1.PC5, U2.MP3_SDI
- new net VBAT: S1.1, U3.VBAT@10
- new net VUSB: N1.VUSB@2, U3.VUSB
- net 5.5V: now also C1.2, J2.VIN, N1.VIN@15, U2.VIN, U3.5.5V@3, U3.5.5V@8, U4.EN, U4.VIN; no longer C17.2, C25.1, C28.1, C45.1, J4.VIN, P7.1, P8.1, R4.2, U12.EN, U12.VIN, U2.VOUT, U7.EN, U7.VIN, U8.EN, U8.VIN
- net GND: now also C1.1, C2.1, C3.2, C4.2, N1.GND@1, N1.GND@16, U1.A0, U1.A1, U1.GND, U1.PAD, U2.GND@1, U2.GND@3, U3.GND@5, U3.GND@9, U4.GND; no longer BATT(VCC-GND).2, C1.2, C10.1, C11.2, C15.1, C16.1, C17.1, C18.1, C2.2, C20.1, C21.1, C22.1, C23.1, C24.1, C25.2, C26.2, C27.2, C28.2, C29.2, C30.1, C31.1, C32.1, C33.1, C34.1, C35.1, C37.1, C38.1, C39.1, C42.2, C43.2, C44.1, C45.2, C46.2, C47.1, C50.1, C6.1, C7.1, C8.2, C9.1, D4.2, D5.2, J1.DET_B, J2.SHIELD@1, J2.SHIELD@2, J2.SHIELD@3, J2.SHIELD@4, J2.SHIELD@5, J2.SHIELD@6, J3.SLEEVE, J4.GND, P7.3, P8.3, P9.2, R12.2, R18.2, R19.1, R3.2, R5.2, U1.GND@23, U1.GND@47, U1.GNDA, U10.AGND, U11.GND, U12.GND, U13.A0, U13.A1, U13.GND, U13.PAD, U2.GND, U2.PAD, U2.PAD0, U2.PAD1, U2.PAD2, U2.PAD3, U2.PGND, U3.GND@3, U4.AGND, U4.GND@17, U4.GND@20, U4.GND@4, U4.GND@PAD, U4.TEST, U5.GND, U6.GND, U7.GND, U8.GND, U9.SCANEN, U9.VSS_1, U9.VSS_2, U9.VSS_3, U9.VSS_4, U9.VSS_5, X1.GND0, X1.GND1, X2.GND0, X2.GND1
- net I2C_SCL: now also J2.CLK, N1.PC0/SCL, R1.1, U1.SCL, U2.I2C_SCL; no longer J4.CLK, P2.2, R20.2, U1.PB6, U13.SCL, U9.SCL
- net I2C_SDA: now also J2.DATA, N1.PC1/SDA, R2.1, U1.SDA, U2.I2C_SDA; no longer J4.DATA, P2.3, R21.2, U1.PB7, U13.SDA, U9.SDA
- net MICROSD_MISO: now also N1.PB0; no longer U1.PB12
- net MICROSD_MOSI: now also N1.PB2; no longer U1.PB14
- net MICROSD_SCK: now also N1.PB1; no longer U1.PB13
- net N$1: now also SW1.1, U1.GP0; no longer C27.1, P6.3, U1.!RST
- net N$11: now also S1.3, U3.BOOST_IN; no longer C37.2, R15.1, U9.FILT
- net N$2: now also SW2.1, U1.GP1; no longer C31.2, R11.1, U9.XTI, X2.1
- net N$3: now also SW3.1, U1.GP2; no longer C30.2, R11.2, U9.XTO, X2.2
- net N$4: now also SW4.1, U1.GP3; no longer C9.2, U1.PF0/OSC_IN, X1.2
- net N$5: now also SW5.1, U1.GP4; no longer C10.2, U1.PF1/OSC_OUT, X1.1
- net N$6: now also SW6.1, U1.GP5; no longer C36.1, R13.2, U9.PVDD
- net N$7: now also SW7.1, U1.GP6; no longer C36.2, R12.1, U9.PVSS
- net OLED_RST: now also J2.RST, N1.PD4; no longer J4.RST, U1.PA4
Other:
- note removed: "128x64 Monochrome OLED Provides UI"
- note removed: "Audio Blocks - CS4334 D/A Converter - LM4811 Headphone Amp"
- note removed: "Audio Regulator Provides 5.0V to Audio blocks: - D/A Converter - Headphone Amp"
- note removed: "Boost Circuit Pumps up Battery Voltage to 5.5V"
- note removed: "CS4334 DAC Converts Digital Audio from STA013 Feeds Analog Audio to Headphone Amplifier"
- note removed: "Charge Circuit Charges Single-Cell LiPo from USB Provides input to Boost Circuit"
- note removed: "Core Logic Blocks Includes - STM32F030 Microcontroller - STA013 MP3 Decoder"
- note removed: "Core Regulator Provides 3.3V to Core Logic blocks: - STM32F030 - STA013"
- note removed: "LM4811 Headphone Amplifier Provides Volume Control"
- note removed: "MCP23008 I/O Expander Provides Button Interface"
- note removed: "MicroSD Adapter Exposes SPI Interface to STM32F0"
- note removed: "MicroSD Block Includes uSD Card reader"
- note removed: "MicroSD Regulator Provides 3.3V to the MicroSD Card"
- note removed: "STA013 MP3 Decoder Provides Digital Audio Output to DAC"
- note removed: "UI Blocks - 128x64 Monochrome OLED - MCP23008 I/O Expander + 7 Buttons"
- note removed: "USB & Power Blocks Include USB LiPo Charger Provides USB UART"
- note removed: "USB UART Circuit Provides USB Serial Interface"
- note removed: "USB-Serial Level Switcher Bridges FT232R UART (5V) with STM32F0 UART (3.3V)"
- moved on the sheet: C1, C2, C5, J1, R1, R2, SW1, SW2, SW3, SW4, SW5, SW6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

Commit message: Finished Shiva board
Connections:
- net MICROSD_CS: now also N1.PB0; no longer N1.PB3
- net MICROSD_MISO: now also N1.PB3; no longer N1.PB0
- net MICROSD_MOSI: now also N1.PB1; no longer N1.PB2
- net MICROSD_SCK: now also N1.PB2; no longer N1.PB1
Changed lines of the file:
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@@
 </segment>
 <segment>
-<pinref part="N1" gate="N1" pin="PB0"/>
-<wire x1="35.56" y1="213.36" x2="-10.16" y2="213.36" width="0.1524" layer="91"/>
-<label x="-7.62" y="213.36" size="1.778" layer="95"/>
+<pinref part="N1" gate="N1" pin="PB3"/>
+<wire x1="35.56" y1="198.12" x2="-10.16" y2="198.12" width="0.1524" layer="91"/>
+<label x="-7.62" y="198.12" size="1.778" layer="95"/>
 </segment>
 </net>
@@
 </segment>
 <segment>
-<pinref part="N1" gate="N1" pin="PB1"/>
-<wire x1="35.56" y1="208.28" x2="-10.16" y2="208.28" width="0.1524" layer="91"/>
-<label x="-7.62" y="208.28" size="1.778" layer="95"/>
+<pinref part="N1" gate="N1" pin="PB2"/>
+<wire x1="35.56" y1="203.2" x2="-10.16" y2="203.2" width="0.1524" layer="91"/>
+<label x="-7.62" y="203.2" size="1.778" layer="95"/>
 </segment>
 </net>
@@
 </segment>
 <segment>
-<pinref part="N1" gate="N1" pin="PB2"/>
-<wire x1="35.56" y1="203.2" x2="-10.16" y2="203.2" width="0.1524" layer="91"/>
-<label x="-7.62" y="203.2" size="1.778" layer="95"/>
+<pinref part="N1" gate="N1" pin="PB1"/>
+<wire x1="35.56" y1="208.28" x2="-10.16" y2="208.28" width="0.1524" layer="91"/>
+<label x="-7.62" y="208.28" size="1.778" layer="95"/>
 </segment>
 </net>
@@
 </segment>
 <segment>
-<pinref part="N1" gate="N1" pin="PB3"/>
-<wire x1="35.56" y1="198.12" x2="-10.16" y2="198.12" width="0.1524" layer="91"/>
-<label x="-7.62" y="198.12" size="1.778" layer="95"/>
+<pinref part="N1" gate="N1" pin="PB0"/>
+<wire x1="35.56" y1="213.36" x2="-10.16" y2="213.36" width="0.1524" layer="91"/>
+<label x="-7.62" y="213.36" size="1.778" layer="95"/>
 </segment>
 </net>
