File: eagle/proj/Dooba/ionode.sch (EAGLE design)
At the start: 25 parts, among them P1 PIN_2, P2 PIN_2, P3 PIN_2, P4 PIN_2, U1 ATMEGA328PB32-VQFN, U2 LP3985SOT23-5, U3 MIC550XSOT23, U4 WRL-13678WRL-13678-QUIET, U5 SN74LVC1G125SOT23-5, U6 SN74LVC1G125SOT23-5, X1 20MHz

Commit message: Redesigned ioNode using ATMEGA1284P, replaced esp8266 with ft232rq usb/serial
Parts:
- removed C5, C6, C7, C8: 1uF, dooba:CAP0805
- removed IO[0-7], IO[8-15]: PIN_8, dooba:PIN_8
- removed P1, P2, P3, P4: PIN_2, dooba:PIN_2
- removed U2: LP3985SOT23-5, dooba:LP3985SOT23-5
- removed U3: MIC550XSOT23, dooba:MIC550XSOT23
- added C21, C22: 10uF, dooba:CAP0805
- added C23, C24: 100nF, dooba:CAP0805
- added C25, C26: 1uF, dooba:CAP0805
- added D3: TX, dooba:LED0805
- added D4: PWR, dooba:LED0805
- added ICSP(MOSI-MISO-SCK-RST-GND): PIN_5, dooba:PIN_5
- added J2: USB-BAMPHENOL-MICRO, dooba:USB-BAMPHENOL-MICRO
- added PA[0-3]/ADC[0-3], PA[4-7]/ADC[4-7], PB[0-3], PC[4-7], PC[O-3](SCL-SDA-PC2-PC3), PD[4-7]: PIN_4, dooba:PIN_4
- added R10, R9: 1k, dooba:RES0805
- added U7: 3.3V, dooba:LP3985SOT23-5
- added VIN-GND, VUSB-GND: PIN_2, dooba:PIN_2
- D2: value PWR -> RX
- R2, R3: value 330R -> 1k
- U1: value ATMEGA328PB32-VQFN -> ATMEGA1284P-MU44-VQFN; device dooba:ATMEGA328PB32-VQFN -> dooba:ATMEGA1284P-MU44-VQFN
- U4: value WRL-13678WRL-13678-QUIET -> FT232RQFN32; device dooba:WRL-13678WRL-13678-QUIET -> dooba:FT232RQFN32
- X1: value 20MHz -> 10MHz
Connections:
- net N$12 renamed ATMEGA_RX
- net N$13 renamed ATMEGA_TX
- removed net N$10: C6.1, P4.2, U3.VOUT, U4.!RST, U4.CHPD, U4.VCC, U6.!OE, U6.VCC
- removed net N$11: U4.TX, U5.A
- removed net N$14: P1.1, U1.PB3/MOSI
- removed net N$15: P2.2, U1.PB4/MISO
- removed net N$16: P2.1, U1.PB5/SCK
- removed net N$17: IO[0-7].2, U1.PD3
- removed net N$18: IO[0-7].3, U1.PD4
- removed net N$19: IO[0-7].4, U1.PE1
- removed net N$20: IO[0-7].5, U1.PD5
- removed net N$28: IO[8-15].5, U1.PC2/ADC2
- removed net N$29: IO[8-15].6, U1.PC3/ADC3
- removed net N$30: IO[8-15].7, U1.PC4/ADC4
- removed net N$31: IO[8-15].8, U1.PC5/ADC5
- removed net N$4: P1.2, R1.2, U1.PC6/!RST
- removed net N$7: D1.1, R3.2
- removed net N$8: C1.2, U1.PB6/XTAL1, X1.2
- removed net N$9: C2.2, U1.PB7/XTAL2, X1.1
- removed net VCC: C3.2, C5.1, P3.1, R1.1, R2.2, U1.AREF, U1.AVCC, U1.VCC, U2.VOUT, U5.!OE, U5.VCC
- new net !RESET: ICSP(MOSI-MISO-SCK-RST-GND).4, R1.2, U1.!RESET
- new net 3.3V: C26.1, C3.1, R1.1, R3.2, U1.AREF, U1.AVCC, U1.VCC@17, U1.VCC@38, U1.VCC@5, U5.!OE, U5.VCC, U7.VOUT
- new net FT232R_RX: U4.RXD, U6.Y
- new net FT232R_TX: U4.TXD, U5.A
- new net PA0/ADC0: PA[0-3]/ADC[0-3].1, U1.PA0/ADC0
- new net PA1/ADC1: PA[0-3]/ADC[0-3].2, U1.PA1/ADC1
- new net PA2/ADC2: PA[0-3]/ADC[0-3].3, U1.PA2/ADC2
- new net PA3/ADC3: PA[0-3]/ADC[0-3].4, U1.PA3/ADC3
- new net PA4/ADC4: PA[4-7]/ADC[4-7].1, U1.PA4/ADC4
- new net PA5/ADC5: PA[4-7]/ADC[4-7].2, U1.PA5/ADC5
- new net PA6/ADC6: PA[4-7]/ADC[4-7].3, U1.PA6/ADC6
- new net PA7/ADC7: PA[4-7]/ADC[4-7].4, U1.PA7/ADC7
- new net PB0: PB[0-3].1, U1.PB0
- new net PB1: PB[0-3].2, U1.PB1
- new net PB2: PB[0-3].3, U1.PB2
- new net PB3: PB[0-3].4, U1.PB3
- new net PB5/MOSI: ICSP(MOSI-MISO-SCK-RST-GND).1, U1.PB5/MOSI
- new net PB6/MISO: ICSP(MOSI-MISO-SCK-RST-GND).2, U1.PB6/MISO
- new net PB7/SCK: ICSP(MOSI-MISO-SCK-RST-GND).3, U1.PB7/SCK
- new net PC0/SCL: PC[O-3](SCL-SDA-PC2-PC3).1, U1.PC0/SCL
- new net PC1/SDA: PC[O-3](SCL-SDA-PC2-PC3).2, U1.PC1/SDA
- new net PC2: PC[O-3](SCL-SDA-PC2-PC3).3, U1.PC2
- new net PC3: PC[O-3](SCL-SDA-PC2-PC3).4, U1.PC3
- new net PC4: PC[4-7].1, U1.PC4
- new net PC5: PC[4-7].2, U1.PC5
- new net PC6: PC[4-7].3, U1.PC6
- new net PC7: PC[4-7].4, U1.PC7
- new net PD2/RXD1: U1.PD2/RXD1
- new net PD3/TXD1: U1.PD3/TXD1
- new net PD4: PD[4-7].1, U1.PD4
- new net PD5: PD[4-7].2, U1.PD5
- new net PD6: PD[4-7].3, U1.PD6
- new net PD7: PD[4-7].4, U1.PD7
- new net VIN: C25.1, U7.EN, U7.VIN, VIN-GND.1
- new net VUSB: C21.2, C22.2, C23.2, J2.VCC, R10.1, R9.1, U4.!RESET, U4.VCC, U4.VCCIO, U6.!OE, U6.VCC, VUSB-GND.1
- net GND: now also C21.1, C22.1, C23.1, C24.1, C25.2, C26.2, C3.2, D4.2, ICSP(MOSI-MISO-SCK-RST-GND).5, J2.GND, J2.SHIELD@1, J2.SHIELD@2, J2.SHIELD@3, J2.SHIELD@4, J2.SHIELD@5, J2.SHIELD@6, U1.GND@18, U1.GND@28, U1.GND@39, U1.GND@6, U1.PAD, U4.AGND, U4.GND@17, U4.GND@20, U4.GND@4, U4.GND@PAD, U4.TEST, U7.GND, VIN-GND.2, VUSB-GND.2; no longer C3.1, C5.2, C6.2, C7.2, C8.2, D2.2, P4.1, U1.GND@21, U1.GND@5, U1.GND@PAD, U2.GND, U3.GND, U4.GND
- net N$1: now also C2.2, U1.XTAL2, X1.2; no longer C7.1, C8.1, P3.2, U2.EN, U2.VIN, U3.EN, U3.VIN
- net N$2: now also C1.2, U1.XTAL1, X1.1; no longer IO[0-7].1, U1.PD2
- net N$21: now also C24.2, U4.3V3OUT; no longer IO[0-7].6, U1.PD6
- net N$22: now also D2.2, U4.CBUS0; no longer IO[0-7].7, U1.PD7
- net N$23: now also D3.2, U4.CBUS1; no longer IO[0-7].8, U1.PB0
- net N$24: now also D2.1, R9.2; no longer IO[8-15].1, U1.PB1
- net N$25: now also D3.1, R10.2; no longer IO[8-15].2, U1.PB2
- net N$26: now also J2.D-, U4.USBDM; no longer IO[8-15].3, U1.PC0/ADC0
- net N$27: now also J2.D+, U4.USBDP; no longer IO[8-15].4, U1.PC1/ADC1
- net N$3: now also D4.1, R3.1; no longer D2.1, R2.1
- net N$5: now also D1.1, R2.1; no longer U4.RX, U6.Y
- net N$6: now also R2.2, U1.PB4; no longer R3.1, U1.PE0
Other:
- note added: "Core Regulator Provides 3.3V to Core Logic blocks: - STM32F030 - STA013"
- note added: "USB UART Circuit Provides USB Serial Interface"
- note added: "USB-Serial Level Switcher Bridges FT232R UART (5V) with STM32F0 UART (3.3V)"
- moved on the sheet: C1, C2, C3, D1, D2, R1, R2, R3, U5, U6, X1

Commit message: Started designing Shiva mp3 player (new version)
Other:
- note removed: "Core Regulator Provides 3.3V to Core Logic blocks: - STM32F030 - STA013"
- note removed: "USB UART Circuit Provides USB Serial Interface"
- note removed: "USB-Serial Level Switcher Bridges FT232R UART (5V) with STM32F0 UART (3.3V)"
Changed lines of the file:
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@@
 <sheet>
 <plain>
-<wire x1="182.88" y1="180.34" x2="182.88" y2="55.88" width="0.1524" layer="97"/>
-<wire x1="182.88" y1="55.88" x2="7.62" y2="55.88" width="0.1524" layer="97"/>
-<wire x1="7.62" y1="55.88" x2="7.62" y2="180.34" width="0.1524" layer="97"/>
-<wire x1="7.62" y1="180.34" x2="182.88" y2="180.34" width="0.1524" layer="97"/>
-<text x="12.7" y="172.72" size="1.778" layer="97">USB UART Circuit
-Provides USB Serial Interface</text>
-<wire x1="152.4" y1="190.5" x2="152.4" y2="246.38" width="0.1524" layer="97"/>
-<wire x1="152.4" y1="246.38" x2="78.74" y2="246.38" width="0.1524" layer="97"/>
-<wire x1="78.74" y1="246.38" x2="78.74" y2="190.5" width="0.1524" layer="97"/>
-<wire x1="78.74" y1="190.5" x2="152.4" y2="190.5" width="0.1524" layer="97"/>
-<text x="149.86" y="198.12" size="1.778" layer="97" rot="R180">USB-Serial Level Switcher
-Bridges FT232R UART (5V) with STM32F0 UART (3.3V)</text>
-<wire x1="294.64" y1="256.54" x2="368.3" y2="256.54" width="0.1524" layer="97"/>
-<wire x1="368.3" y1="256.54" x2="368.3" y2="200.66" width="0.1524" layer="97"/>
-<wire x1="368.3" y1="200.66" x2="294.64" y2="200.66" width="0.1524" layer="97"/>
-<wire x1="294.64" y1="200.66" x2="294.64" y2="256.54" width="0.1524" layer="97"/>
-<text x="297.18" y="243.84" size="1.778" layer="97">Core Regulator
-Provides 3.3V to Core Logic blocks:
- - STM32F030
- - STA013</text>
-<wire x1="287.02" y1="175.26" x2="287.02" y2="12.7" width="0.1524" layer="97"/>
-<wire x1="287.02" y1="12.7" x2="502.92" y2="12.7" width="0.1524" layer="97"/>
-<wire x1="502.92" y1="12.7" x2="502.92" y2="175.26" width="0.1524" layer="97"/>
-<wire x1="502.92" y1="175.26" x2="287.02" y2="175.26" width="0.1524" layer="97"/>
 </plain>
 <instances>
@@
 </schematic>
 </drawing>
-<compatibility>
-<note version="6.3" minversion="6.2.2" severity="warning">
-Since Version 6.2.2 text objects can contain more than one line,
-which will not be processed correctly with this version.
-</note>
-</compatibility>
 </eagle>

Commit message: Fixed STA013 Device in Eagle Library Fixed Aecho Board to use updated STA013 Fixed ioNode Schematic (74125 buffers for USB UART had their !OE tied to VCC...)
Connections:
- net 3.3V: no longer U5.!OE
- net GND: now also U5.!OE, U6.!OE
- net VUSB: no longer U6.!OE
Changed lines of the file:
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@@
 <?xml version="1.0" encoding="utf-8"?>
 <!DOCTYPE eagle SYSTEM "eagle.dtd">
-<eagle version="7.7.0">
+<eagle version="7.3.0">
 <drawing>
 <settings>
@@
 <setting verticaltext="up"/>
 </settings>
-<grid distance="0.1" unitdist="inch" unit="inch" style="lines" multiple="1" display="no" altdistance="0.01" altunitdist="inch" altunit="inch"/>
+<grid distance="0.05" unitdist="inch" unit="inch" style="lines" multiple="1" display="no" altdistance="0.01" altunitdist="inch" altunit="inch"/>
 <layers>
 <layer number="1" name="Top" color="4" fill="1" visible="no" active="no"/>
@@
 <pinref part="GND51" gate="1" pin="GND"/>
 <pinref part="U5" gate="U1" pin="GND"/>
-<wire x1="116.84" y1="236.22" x2="116.84" y2="233.68" width="0.1524" layer="91"/>
+<wire x1="116.84" y1="236.22" x2="116.84" y2="234.95" width="0.1524" layer="91"/>
+<pinref part="U5" gate="U1" pin="!OE"/>
+<wire x1="116.84" y1="234.95" x2="116.84" y2="233.68" width="0.1524" layer="91"/>
+<wire x1="127" y1="233.68" x2="127" y2="234.95" width="0.1524" layer="91"/>
+<wire x1="127" y1="234.95" x2="116.84" y2="234.95" width="0.1524" layer="91"/>
+<junction x="116.84" y="234.95"/>
 </segment>
 <segment>
 <pinref part="U6" gate="U1" pin="GND"/>
 <pinref part="GND52" gate="1" pin="GND"/>
-<wire x1="109.22" y1="208.28" x2="109.22" y2="205.74" width="0.1524" layer="91"/>
+<wire x1="109.22" y1="208.28" x2="109.22" y2="207.01" width="0.1524" layer="91"/>
+<pinref part="U6" gate="U1" pin="!OE"/>
+<wire x1="109.22" y1="207.01" x2="109.22" y2="205.74" width="0.1524" layer="91"/>
+<wire x1="99.06" y1="208.28" x2="99.06" y2="207.01" width="0.1524" layer="91"/>
+<wire x1="99.06" y1="207.01" x2="109.22" y2="207.01" width="0.1524" layer="91"/>
+<junction x="109.22" y="207.01"/>
 </segment>
 <segment>
@@
 <pinref part="U5" gate="U1" pin="VCC"/>
 <wire x1="127" y1="208.28" x2="127" y2="205.74" width="0.1524" layer="91"/>
-<pinref part="U5" gate="U1" pin="!OE"/>
-<wire x1="127" y1="236.22" x2="127" y2="233.68" width="0.1524" layer="91"/>
-<wire x1="127" y1="236.22" x2="132.08" y2="236.22" width="0.1524" layer="91"/>
-<wire x1="132.08" y1="236.22" x2="132.08" y2="205.74" width="0.1524" layer="91"/>
-<wire x1="132.08" y1="205.74" x2="127" y2="205.74" width="0.1524" layer="91"/>
-<wire x1="132.08" y1="205.74" x2="172.72" y2="205.74" width="0.1524" layer="91"/>
-<junction x="132.08" y="205.74"/>
+<wire x1="127" y1="205.74" x2="172.72" y2="205.74" width="0.1524" layer="91"/>
 <label x="170.18" y="205.74" size="1.778" layer="95" rot="R180"/>
 </segment>
@@
 <pinref part="U6" gate="U1" pin="VCC"/>
 <wire x1="99.06" y1="233.68" x2="99.06" y2="236.22" width="0.1524" layer="91"/>
-<wire x1="99.06" y1="236.22" x2="93.98" y2="236.22" width="0.1524" layer="91"/>
-<pinref part="U6" gate="U1" pin="!OE"/>
-<wire x1="99.06" y1="208.28" x2="99.06" y2="205.74" width="0.1524" layer="91"/>
-<wire x1="93.98" y1="236.22" x2="93.98" y2="205.74" width="0.1524" layer="91"/>
-<wire x1="93.98" y1="205.74" x2="99.06" y2="205.74" width="0.1524" layer="91"/>
-<wire x1="93.98" y1="236.22" x2="58.42" y2="236.22" width="0.1524" layer="91"/>
-<junction x="93.98" y="236.22"/>
+<wire x1="99.06" y1="236.22" x2="58.42" y2="236.22" width="0.1524" layer="91"/>
 <label x="76.2" y="236.22" size="1.778" layer="95" rot="R180"/>
 </segment>
