File: proj/stickie.brd (EAGLE design)
At the start: 84.1 x 15.2 mm, 18 parts, among them J1 DM3D-SFDM, P1 PC, P2 PA, P3 PWR_OUT(5.5V-GND), P4 PD6-7, P5 GND, P6 GND, U1 WRL-13678WRL-13678-QUIET, U3 DOOBA_NOMAD, U4 3.3V 500mA

Commit message: Updated stickie board to use SPI for MicroSD @close #8
Connections:
- removed net MICROSD_MISO: J1.DAT0/DO, N1.14
- removed net MICROSD_MOSI: J1.CMD/DI, N1.12
- removed net MICROSD_SCK: J1.CLK/SCK, N1.13
- new net SPI_MISO: J1.DAT0/DO, N1.32
- new net SPI_MOSI: J1.CMD/DI, N1.31
- new net SPI_SCK: J1.CLK/SCK, N1.33
Routing:
- net MICROSD_MOSI: track 41.2 -> 0.00 mm, vias 1 -> 0
- net MICROSD_SCK: track 36.0 -> 0.00 mm, vias 1 -> 0
- net MICROSD_MISO: track 30.8 -> 0.00 mm, vias 1 -> 0
- net SPI_MOSI: track 0.00 -> 29.3 mm, vias 0 -> 1
- net SPI_SCK: track 0.00 -> 25.5 mm, vias 0 -> 1
- net SPI_MISO: track 0.00 -> 23.8 mm, vias 0 -> 1
- net WIFI_FLASH: track 54.3 -> 55.6 mm
- net 5.5V: track 84.2 -> 83.0 mm, vias 0 -> 2
- net WIFI_RX: track 41.2 -> 42.2 mm
- net MICROSD_CS: track 45.2 -> 45.9 mm
