File: proj/stickie.sch (EAGLE design)
At the start: 18 parts, among them J1 DM3D-SFDM, P1 PC, P2 PA, P3 PWR_OUT(5.5V-GND), P4 PD6-7, P5 GND, P6 GND, U1 WRL-13678WRL-13678-QUIET, U3 DOOBA_NOMAD, U4 3.3V 500mA

Commit message: Updated stickie board to use SPI for MicroSD @close #8
Connections:
- removed net MICROSD_MISO: J1.DAT0/DO, N1.PB3
- removed net MICROSD_MOSI: J1.CMD/DI, N1.PB1
- removed net MICROSD_SCK: J1.CLK/SCK, N1.PB2
- new net SPI_MISO: J1.DAT0/DO, N1.MISO
- new net SPI_MOSI: J1.CMD/DI, N1.MOSI
- new net SPI_SCK: J1.CLK/SCK, N1.SCK
Changed lines of the file:
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@@
-</segment>
-</net>
-<net name="MICROSD_MISO" class="0">
-<segment>
-<pinref part="J1" gate="J1" pin="DAT0/DO"/>
-<wire x1="261.62" y1="148.59" x2="193.04" y2="148.59" width="0.1524" layer="91"/>
-<label x="195.58" y="148.59" size="1.778" layer="95"/>
-</segment>
-<segment>
-<wire x1="73.66" y1="121.92" x2="27.94" y2="121.92" width="0.1524" layer="91"/>
-<label x="30.48" y="121.92" size="1.778" layer="95"/>
-<pinref part="N1" gate="N1" pin="PB3"/>
-</segment>
-</net>
-<net name="MICROSD_SCK" class="0">
-<segment>
-<pinref part="J1" gate="J1" pin="CLK/SCK"/>
-<wire x1="261.62" y1="158.75" x2="193.04" y2="158.75" width="0.1524" layer="91"/>
-<label x="195.58" y="158.75" size="1.778" layer="95"/>
-</segment>
-<segment>
-<wire x1="73.66" y1="127" x2="27.94" y2="127" width="0.1524" layer="91"/>
-<label x="30.48" y="127" size="1.778" layer="95"/>
-<pinref part="N1" gate="N1" pin="PB2"/>
-</segment>
-</net>
-<net name="MICROSD_MOSI" class="0">
-<segment>
-<pinref part="J1" gate="J1" pin="CMD/DI"/>
-<wire x1="261.62" y1="168.91" x2="193.04" y2="168.91" width="0.1524" layer="91"/>
-<label x="195.58" y="168.91" size="1.778" layer="95"/>
-</segment>
-<segment>
-<wire x1="73.66" y1="132.08" x2="27.94" y2="132.08" width="0.1524" layer="91"/>
-<label x="30.48" y="132.08" size="1.778" layer="95"/>
-<pinref part="N1" gate="N1" pin="PB1"/>
 </segment>
 </net>
@@
 </segment>
 </net>
+<net name="SPI_SCK" class="0">
+<segment>
+<pinref part="N1" gate="N1" pin="SCK"/>
+<wire x1="93.98" y1="101.6" x2="93.98" y2="96.52" width="0.1524" layer="91"/>
+<wire x1="93.98" y1="96.52" x2="172.72" y2="96.52" width="0.1524" layer="91"/>
+<label x="154.94" y="96.52" size="1.778" layer="95"/>
+</segment>
+<segment>
+<pinref part="J1" gate="J1" pin="CLK/SCK"/>
+<wire x1="261.62" y1="158.75" x2="193.04" y2="158.75" width="0.1524" layer="91"/>
+<label x="195.58" y="158.75" size="1.778" layer="95"/>
+</segment>
+</net>
+<net name="SPI_MISO" class="0">
+<segment>
+<pinref part="N1" gate="N1" pin="MISO"/>
+<wire x1="88.9" y1="101.6" x2="88.9" y2="91.44" width="0.1524" layer="91"/>
+<wire x1="88.9" y1="91.44" x2="172.72" y2="91.44" width="0.1524" layer="91"/>
+<label x="154.94" y="91.44" size="1.778" layer="95"/>
+</segment>
+<segment>
+<pinref part="J1" gate="J1" pin="DAT0/DO"/>
+<wire x1="261.62" y1="148.59" x2="193.04" y2="148.59" width="0.1524" layer="91"/>
+<label x="195.58" y="148.59" size="1.778" layer="95"/>
+</segment>
+</net>
+<net name="SPI_MOSI" class="0">
+<segment>
+<pinref part="N1" gate="N1" pin="MOSI"/>
+<wire x1="83.82" y1="101.6" x2="83.82" y2="86.36" width="0.1524" layer="91"/>
+<wire x1="83.82" y1="86.36" x2="172.72" y2="86.36" width="0.1524" layer="91"/>
+<label x="154.94" y="86.36" size="1.778" layer="95"/>
+</segment>
+<segment>
+<pinref part="J1" gate="J1" pin="CMD/DI"/>
+<wire x1="261.62" y1="168.91" x2="193.04" y2="168.91" width="0.1524" layer="91"/>
+<label x="195.58" y="168.91" size="1.778" layer="95"/>
+</segment>
+</net>
