File: proj/tako.sch (EAGLE design)
At the start: 22 parts, among them U1 ENC28J6028QFN, U2 ARJC02-111008B, X1 25MHz

Commit message: Started designing Tako schematic & board @open #11
Parts:
- added P1: RESET-INT-GND-VIN, dooba:PIN_4
- added P2: SO-SI-SCK-CS, dooba:PIN_4
Connections:
- removed net N$7: R2.1, U1.!CS
- new net !WNC28J60_CS: P2.4, R2.1, U1.!CS
- net !ENC28J60_RESET: now also P1.1
- net ENC28J60_INT: now also P1.2
- net ENC28J60_SCK: now also P2.3
- net ENC28J60_SI: now also P2.2
- net ENC28J60_SO: now also P2.1
- net GND: now also P1.3
- net VIN: now also P1.4
Changed lines of the file:
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@@
 <part name="GND23" library="supply1" deviceset="GND" device=""/>
 <part name="GND24" library="supply1" deviceset="GND" device=""/>
+<part name="P1" library="dooba" deviceset="PIN_4" device="" value="RESET-INT-GND-VIN"/>
+<part name="P2" library="dooba" deviceset="PIN_4" device="" value="SO-SI-SCK-CS"/>
+<part name="GND25" library="supply1" deviceset="GND" device=""/>
 </parts>
 <sheets>
@@
 <instance part="GND23" gate="1" x="160.02" y="134.62" rot="R180"/>
 <instance part="GND24" gate="1" x="99.06" y="99.06" rot="R270"/>
+<instance part="P1" gate="P1" x="60.96" y="17.78" rot="R270"/>
+<instance part="P2" gate="P1" x="86.36" y="17.78" rot="R270"/>
+<instance part="GND25" gate="1" x="55.88" y="35.56" rot="R180"/>
 </instances>
 <busses>
@@
 <wire x1="17.78" y1="111.76" x2="17.78" y2="127" width="0.1524" layer="91"/>
 <junction x="17.78" y="127"/>
-<wire x1="17.78" y1="127" x2="-12.7" y2="127" width="0.1524" layer="91"/>
-<label x="-10.16" y="127" size="1.778" layer="95"/>
+<wire x1="17.78" y1="127" x2="5.08" y2="127" width="0.1524" layer="91"/>
+<label x="7.62" y="127" size="1.778" layer="95"/>
+</segment>
+<segment>
+<pinref part="P1" gate="P1" pin="4"/>
+<wire x1="53.34" y1="25.4" x2="53.34" y2="30.48" width="0.1524" layer="91"/>
+<wire x1="53.34" y1="30.48" x2="5.08" y2="30.48" width="0.1524" layer="91"/>
+<label x="7.62" y="30.48" size="1.778" layer="95"/>
 </segment>
 </net>
@@
 <wire x1="101.6" y1="99.06" x2="109.22" y2="99.06" width="0.1524" layer="91"/>
 </segment>
+<segment>
+<pinref part="P1" gate="P1" pin="3"/>
+<pinref part="GND25" gate="1" pin="GND"/>
+<wire x1="55.88" y1="33.02" x2="55.88" y2="25.4" width="0.1524" layer="91"/>
+</segment>
 </net>
 <net name="N$1" class="0">
@@
 </segment>
 </net>
-<net name="N$7" class="0">
+<net name="!WNC28J60_CS" class="0">
 <segment>
 <pinref part="U1" gate="U1" pin="!CS"/>
 <pinref part="R2" gate="R1" pin="1"/>
-<wire x1="134.62" y1="38.1" x2="134.62" y2="53.34" width="0.1524" layer="91"/>
+<wire x1="134.62" y1="38.1" x2="134.62" y2="40.64" width="0.1524" layer="91"/>
+<wire x1="134.62" y1="40.64" x2="134.62" y2="53.34" width="0.1524" layer="91"/>
+<wire x1="134.62" y1="40.64" x2="78.74" y2="40.64" width="0.1524" layer="91"/>
+<junction x="134.62" y="40.64"/>
+<label x="7.62" y="40.64" size="1.778" layer="95"/>
+<pinref part="P2" gate="P1" pin="4"/>
+<wire x1="78.74" y1="40.64" x2="5.08" y2="40.64" width="0.1524" layer="91"/>
+<wire x1="78.74" y1="25.4" x2="78.74" y2="40.64" width="0.1524" layer="91"/>
+<junction x="78.74" y="40.64"/>
 </segment>
 </net>
@@
 <segment>
 <pinref part="U1" gate="U1" pin="!INT"/>
-<wire x1="109.22" y1="88.9" x2="-12.7" y2="88.9" width="0.1524" layer="91"/>
-<label x="-10.16" y="88.9" size="1.778" layer="95"/>
+<wire x1="109.22" y1="88.9" x2="58.42" y2="88.9" width="0.1524" layer="91"/>
+<label x="7.62" y="88.9" size="1.778" layer="95"/>
+<pinref part="P1" gate="P1" pin="2"/>
+<wire x1="58.42" y1="88.9" x2="5.08" y2="88.9" width="0.1524" layer="91"/>
+<wire x1="58.42" y1="25.4" x2="58.42" y2="88.9" width="0.1524" layer="91"/>
+<junction x="58.42" y="88.9"/>
 </segment>
 </net>
@@
 <segment>
 <pinref part="U1" gate="U1" pin="SO"/>
-<wire x1="109.22" y1="78.74" x2="-12.7" y2="78.74" width="0.1524" layer="91"/>
-<label x="-10.16" y="78.74" size="1.778" layer="95"/>
+<label x="7.62" y="78.74" size="1.778" layer="95"/>
+<wire x1="109.22" y1="78.74" x2="86.36" y2="78.74" width="0.1524" layer="91"/>
+<pinref part="P2" gate="P1" pin="1"/>
+<wire x1="86.36" y1="78.74" x2="5.08" y2="78.74" width="0.1524" layer="91"/>
+<wire x1="86.36" y1="25.4" x2="86.36" y2="78.74" width="0.1524" layer="91"/>
+<junction x="86.36" y="78.74"/>
 </segment>
 </net>
@@
 <segment>
 <pinref part="U1" gate="U1" pin="SI"/>
-<wire x1="109.22" y1="73.66" x2="-12.7" y2="73.66" width="0.1524" layer="91"/>
-<label x="-10.16" y="73.66" size="1.778" layer="95"/>
+<label x="7.62" y="73.66" size="1.778" layer="95"/>
+<wire x1="109.22" y1="73.66" x2="83.82" y2="73.66" width="0.1524" layer="91"/>
+<pinref part="P2" gate="P1" pin="2"/>
+<wire x1="83.82" y1="73.66" x2="5.08" y2="73.66" width="0.1524" layer="91"/>
+<wire x1="83.82" y1="25.4" x2="83.82" y2="73.66" width="0.1524" layer="91"/>
+<junction x="83.82" y="73.66"/>
 </segment>
 </net>
@@
 <pinref part="U1" gate="U1" pin="SCK"/>
 <wire x1="129.54" y1="53.34" x2="129.54" y2="50.8" width="0.1524" layer="91"/>
-<wire x1="129.54" y1="50.8" x2="-12.7" y2="50.8" width="0.1524" layer="91"/>
-<label x="-10.16" y="50.8" size="1.778" layer="95"/>
+<wire x1="129.54" y1="50.8" x2="81.28" y2="50.8" width="0.1524" layer="91"/>
+<label x="7.62" y="50.8" size="1.778" layer="95"/>
+<pinref part="P2" gate="P1" pin="3"/>
+<wire x1="81.28" y1="50.8" x2="5.08" y2="50.8" width="0.1524" layer="91"/>
+<wire x1="81.28" y1="25.4" x2="81.28" y2="50.8" width="0.1524" layer="91"/>
+<junction x="81.28" y="50.8"/>
 </segment>
 </net>
@@
 <pinref part="U1" gate="U1" pin="!RESET"/>
 <wire x1="139.7" y1="53.34" x2="139.7" y2="45.72" width="0.1524" layer="91"/>
-<wire x1="139.7" y1="45.72" x2="-12.7" y2="45.72" width="0.1524" layer="91"/>
-<label x="-10.16" y="45.72" size="1.778" layer="95"/>
-</segment>
-</net>
+<wire x1="139.7" y1="45.72" x2="60.96" y2="45.72" width="0.1524" layer="91"/>
+<label x="7.62" y="45.72" size="1.778" layer="95"/>
+<pinref part="P1" gate="P1" pin="1"/>
+<wire x1="60.96" y1="45.72" x2="5.08" y2="45.72" width="0.1524" layer="91"/>
+<wire x1="60.96" y1="25.4" x2="60.96" y2="45.72" width="0.1524" layer="91"/>
+<junction x="60.96" y="45.72"/>
+</segment>
+</net>
