File: proj/fiddle.sch (EAGLE design)
At the start: 12 parts, among them SW6 TACTSW_2MICRO3X6, SW7 TACTSW_2MICRO3X6, U1 MCP23008QFN, U4 3.3V

Commit message: Moved 0.91 OLED footprint to docu layer Updated Fiddle schematic & board to include MicroSD and Wifi (esp8266) :D
Parts:
- added C10, C11, C12, C4, C5, C8, C9: 10uF, dooba:CAP0805
- added C6, C7: 100nF, dooba:CAP0805
- added J1: DM3D-SFDM, dooba:DM3D-SFDM
- added RST: TACTSW_2MICRO3X6, dooba:TACTSW_2MICRO3X6
- added U2: WRL-13678WRL-13678-QUIET, dooba:WRL-13678WRL-13678-QUIET
- U4: value 3.3V -> 3.3V 600mA
Connections:
- new net MICROSD_CS: J1.DAT3/CS, N1.PB3
- new net N$8: N1.!RST, RST.2
- new net SPI_MISO: J1.DAT0/DO, N1.MISO
- new net SPI_MOSI: J1.CMD/DI, N1.MOSI
- new net SPI_SCK: J1.CLK/SCK, N1.SCK
- new net WIFI_FLASH: N1.PD5, U2.GPIO0
- new net WIFI_RST: N1.PD4, U2.!RST
- new net WIFI_RX: N1.PD2/RXD1, U2.TX
- new net WIFI_TX: N1.PD3/TXD1, U2.RX
- net 3.3V: now also C10.1, C11.1, C12.1, C4.1, C5.1, C6.1, C7.1, C8.1, C9.1, J1.VCC, U2.CHPD, U2.VCC
- net GND: now also C10.2, C11.2, C12.2, C4.2, C5.2, C6.2, C7.2, C8.2, C9.2, J1.GND, J1.GND_1, J1.GND_2, J1.GND_3, J1.GND_4, RST.1, U2.GND
