File: proj/fiddle.old.sch (EAGLE design)
At the start: 31 parts, among them J1 DM3D-SFDM, P1 PIN_8, P2 PIN_8, P3 PIN_4, P4 PIN_4, P5 PIN_2, P6 PIN_3, P7 PIN_1, SW6 TACTSW_2MICRO3X6, SW7 TACTSW_2MICRO3X6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

Commit message: tootoot
Parts:
- removed P1, P2: PIN_8, dooba:PIN_8
- removed P3, P4: PIN_4, dooba:PIN_4
- removed P5: PIN_2, dooba:PIN_2
- removed P6: PIN_3, dooba:PIN_3
- removed P7: PIN_1, dooba:PIN_1
Connections:
- removed net N$10: N1.PC6, P2.7
- removed net N$11: N1.PC5, P2.6
- removed net N$12: N1.PC4, P2.5
- removed net N$13: N1.PC3, P2.4
- removed net N$14: N1.PC2, P2.3
- removed net N$15: N1.PA7/ADC7, P1.8
- removed net N$16: N1.PA6/ADC6, P1.7
- removed net N$17: N1.PA5/ADC5, P1.6
- removed net N$18: N1.PA4/ADC4, P1.5
- removed net N$19: N1.PA3/ADC3, P1.4
- removed net N$20: N1.PA2/ADC2, P1.3
- removed net N$21: N1.PA1/ADC1, P1.2
- removed net N$22: N1.PA0/ADC0, P1.1
- removed net N$23: N1.PD7, P4.4
- removed net N$24: N1.PD6, P4.3
- removed net N$25: N1.PD5, P4.2
- removed net N$26: N1.PD4, P4.1
- removed net N$27: N1.PB3, P7.1
- removed net N$9: N1.PC7, P2.8
- net 3.3V: no longer P6.3
- net GND: no longer P5.1, P6.1
- net I2C_SCL: no longer P2.1
- net I2C_SDA: no longer P2.2
- net MICROSD_CS: now also N1.PB3; no longer N1.PB2
- net N$8: no longer P3.1
- net SPI_MISO: no longer P3.3
- net SPI_MOSI: no longer P3.2
- net SPI_SCK: no longer P3.4
- net VIN: no longer P6.2
- net VUSB: no longer P5.2
- net WIFI_FLASH: now also N1.PD5; no longer N1.PB0
- net WIFI_RST: now also N1.PD4; no longer N1.PB1
