File: proj/rizon.sch (EAGLE design)
At the start: 27 parts, among them J1 PWRJACK5521, U1 Z8400, U2 AS6C62256PDIP, U3 AS6C62256PDIP, U4 AT28C64BPLCC, U5 AT28C64BPLCC, U6 7432PDIP, U7 7805TO220, U8 7432PDIP, U9 7400PDIP, X1 OSC412.7

Commit message: Added 74374 to library Further designed Rizon Z80 SBC
Parts:
- added U10: 74374PDIP, dooba:74374PDIP
- added U11: 74138PDIP, dooba:74138PDIP
Connections:
- net !RAM_BANK1_CE renamed !HIGH_ADDR
- net !ROM_BANK1_CE renamed !ROM_BANK1
- removed net N$6: U1.!M1
- new net !INT: U1.!INT
- new net !IODEV0: U11.Y0
- new net !IODEV1: U11.Y1
- new net !IODEV2: U11.Y2
- new net !IODEV3: U11.Y3
- new net !IODEV4: U11.Y4
- new net !IODEV5: U11.Y5
- new net !IODEV6: U11.Y6
- new net !IODEV7: U11.Y7
- new net !M1: U1.!M1, U11.G1
- new net !MEM_SELECT_ROM: U6.1Y
- new net !SCR0_ROM_EN: U10.Q0, U6.1B
- net !IORQ: now also U11.!G2A, U11.!G2B
- net ADDR0: now also U11.A
- net ADDR1: now also U11.B
- net ADDR15: now also U6.1A
- net ADDR2: now also U11.C
- net DATA0: now also U10.D0
- net DATA1: now also U10.D1
- net DATA2: now also U10.D2
- net DATA3: now also U10.D3
- net DATA4: now also U10.D4
- net DATA5: now also U10.D5
- net DATA6: now also U10.D6
- net DATA7: now also U10.D7
Other:
- note added: "EEPROM 2 x 8Kb"
- note added: "IO Device Selector"
- note added: "SCR0 - System Control Register 0"
- note added: "SRAM 2 x 32Kb"
- note added: "Z80 CPU"

Commit message: Started designing main board for Rizon Z80 computer
Parts:
- added !IODEV, P1: ADDR, dooba:PIN_16
- added P2: DATA, dooba:PIN_8
- added P3: CTL, dooba:PIN_16
- added P4: PWR, dooba:PIN_4
- added P5: 10k, dooba:PIN_61LINE
- added U12, U13, U14, U15, U17: 74138PDIP, dooba:74138PDIP
- added U16: 7432PDIP, dooba:7432PDIP
- U10: value 74374PDIP -> 74273PDIP; device dooba:74374PDIP -> dooba:74273PDIP
Connections:
- removed net N$7: U9.3Y
- new net !BUSACK: P3.10, U1.!BUSACK
- new net !BUSREQ: P3.12, P5.6, U1.!BUSREQ
- new net !IODEV10: !IODEV.11, U12.Y2
- new net !IODEV11: !IODEV.12, U12.Y3
- new net !IODEV12: !IODEV.13, U12.Y4
- new net !IODEV13: !IODEV.14, U12.Y5
- new net !IODEV14: !IODEV.15, U12.Y6
- new net !IODEV15: !IODEV.16, U12.Y7
- new net !IODEV8: !IODEV.9, U12.Y0
- new net !IODEV9: !IODEV.10, U12.Y1
- new net !IO_SELECT_BANK0: U11.!G2B, U13.Y0
- new net !IO_SELECT_BANK1: U12.!G2B, U13.Y1
- new net !MEM_SELECT_LOWRAM: U6.2Y, U8.1A
- new net !MEM_SELECT_ROM_BANK0: U6.3Y, U8.3A
- new net !MEM_SELECT_ROM_BANK1: U6.4Y, U8.4A
- new net !NMI: P3.4, P5.3, U1.!NMI
- new net !RAM_BANK0_CE: U2.!CE, U8.1Y
- new net !RAM_BANK1_CE: U3.!CE, U8.2Y
- new net !RESET: P3.15, P5.4, U1.!RESET, U10.!MR
- new net !RFSH: P3.14, U1.!RFSH
- new net !ROM_BANK0_CE: U4.!CE, U8.3Y
- new net !ROM_BANK1_CE: U5.!CE, U8.4Y
- new net !SCR0_CP: U16.1Y, U9.4A, U9.4B
- new net !WAIT: P3.11, P5.5, U1.!WAIT
- new net CLK: P3.1, U1.CLK, X1.OUT
- new net N$1: U13.!G2B, U14.Y0
- new net N$2: U14.!G2B, U15.Y0
- new net N$3: U15.!G2B, U17.Y0
- new net N$4: J1.PWR, S1.1, S1.4
- new net SCR0_CP: U10.CP, U9.4Y
- new net SCR0_ROM_EN: U6.2B, U9.3Y
- new net VCC: C1.2, C10.2, C11.2, C12.2, C13.2, C14.2, C15.2, C2.2, C5.2, C6.2, C7.2, C8.2, C9.2, P4.4, P5.1, U1.VCC, U10.VCC, U11.VCC, U12.VCC, U13.VCC, U14.VCC, U15.VCC, U16.VCC, U17.VCC, U2.VCC, U3.VCC, U4.VCC, U5.VCC, U6.VCC, U7.VOUT, U8.VCC, U9.VCC, X1.VCC
- new net VIN: C3.2, C4.2, P4.2, S1.2, S1.5, U7.VIN
- net !HALT: now also P3.5
- net !HIGH_ADDR: now also U8.2A
- net !INT: now also P3.3, P5.2
- net !IODEV0: now also U16.1A
- net !IODEV1: now also !IODEV.2
- net !IODEV2: now also !IODEV.3
- net !IODEV3: now also !IODEV.4
- net !IODEV4: now also !IODEV.5
- net !IODEV5: now also !IODEV.6
- net !IODEV6: now also !IODEV.7
- net !IODEV7: now also !IODEV.8
- net !IORQ: now also P3.7, U12.!G2A, U13.!G2A, U14.!G2A, U15.!G2A, U17.!G2A; no longer U11.!G2B
- net !M1: now also P3.13, U12.G1, U13.G1, U14.G1, U15.G1, U17.G1
- net !MEM_SELECT_ROM: now also U6.3B, U6.4B
- net !MREQ: now also P3.6, U8.1B, U8.2B, U8.3B, U8.4B
- net !RD: now also P3.8, U2.!OE, U3.!OE, U4.!OE, U5.!OE
- net !ROM_BANK1: now also U6.4A
- net !SCR0_ROM_EN: now also U9.3A, U9.3B
- net !WR: now also P3.9, U16.1B, U2.!WE, U3.!WE, U4.!WE, U5.!WE
- net ADDR0: now also P1.1, U12.A
- net ADDR1: now also P1.2, U12.B
- net ADDR10: now also P1.11, U15.B
- net ADDR11: now also P1.12, U15.C
- net ADDR12: now also P1.13, U17.A
- net ADDR13: now also P1.14, U17.B, U6.3A
- net ADDR14: now also P1.15, U17.C
- net ADDR15: now also P1.16, U17.!G2B, U6.2A
- net ADDR2: now also P1.3, U12.C
- net ADDR3: now also P1.4, U13.A
- net ADDR4: now also P1.5, U13.B
- net ADDR5: now also P1.6, U13.C
- net ADDR6: now also P1.7, U14.A
- net ADDR7: now also P1.8, U14.B
- net ADDR8: now also P1.9, U14.C
- net ADDR9: now also P1.10, U15.A
- net DATA0: now also P2.1, U2.DQ0, U3.DQ0, U4.I/O0, U5.I/O0
- net DATA1: now also P2.2, U2.DQ1, U3.DQ1, U4.I/O1, U5.I/O1
- net DATA2: now also P2.3, U2.DQ2, U3.DQ2, U4.I/O2, U5.I/O2
- net DATA3: now also P2.4, U2.DQ3, U3.DQ3, U4.I/O3, U5.I/O3
- net DATA4: now also P2.5, U2.DQ4, U3.DQ4, U4.I/O4, U5.I/O4
- net DATA5: now also P2.6, U2.DQ5, U3.DQ5, U4.I/O5, U5.I/O5
- net DATA6: now also P2.7, U2.DQ6, U3.DQ6, U4.I/O6, U5.I/O6
- net DATA7: now also P2.8, U2.DQ7, U3.DQ7, U4.I/O7, U5.I/O7
- net GND: now also !IODEV.1, P3.16, P3.2, P4.1, P4.3, U10.GND, U11.GND, U12.GND, U13.GND, U14.GND, U15.GND, U16.GND, U17.GND
Other:
- note added: "Address Decoding"
- note added: "Connectors"
- note added: "Memory (RAM + ROM)"
- note added: "Memory Device Selector"
- moved on the sheet: C1, C10, C11, C12, C13, C14, C15, C2, C3, C4, C5, C8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

Commit message: Further designed Rizon board
Connections:
- net !BUSACK: now also P3.7; no longer P3.10
- net !BUSREQ: now also P3.2; no longer P3.12
- net !HALT: now also P3.10; no longer P3.5
- net !INT: now also P3.12; no longer P3.3
- net !IORQ: now also P3.8, U12.!G2B; no longer P3.7, U12.!G2A
- net !IO_SELECT_BANK1: now also U12.!G2A; no longer U12.!G2B
- net !M1: now also P3.1; no longer P3.13
- net !MREQ: now also P3.11; no longer P3.6
- net !NMI: now also P3.13; no longer P3.4
- net !RD: now also P3.9; no longer P3.8
- net !RESET: now also P3.3, P5.5; no longer P3.15, P5.4
- net !RFSH: now also P3.5; no longer P3.14
- net !WAIT: now also P3.4, P5.4; no longer P3.11, P5.5
- net !WR: now also P3.6; no longer P3.9
- net CLK: now also P3.15; no longer P3.1
- net GND: now also P3.14; no longer P3.2
