File: proj/rizon-bckp.sch (EAGLE design)
At the start: 32 parts, among them J1 PWRJACK5521, P1 ADDR, P2 DATA, P3 CTL, P4 PWR, P5 10k, U1 Z8400, U2 AS6C62256PDIP, U3 AS6C62256PDIP, U4 AT28C64BPLCC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

Commit message: Redesigning Rizon board
Parts:
- added !IODEV: ADDR, dooba:PIN_16
- added U10: 74273PDIP, dooba:74273PDIP
- added U11, U12, U13, U14, U15, U17: 74138PDIP, dooba:74138PDIP
- added U16: 7432PDIP, dooba:7432PDIP
Connections:
- net ROM_EN renamed SCR0_ROM_EN
- removed net !ROM_EN: P3.14, U6.1B, U9.3A, U9.3B
- new net !IODEV0: U11.Y0, U16.1A
- new net !IODEV1: !IODEV.2, U11.Y1
- new net !IODEV10: !IODEV.11, U12.Y2
- new net !IODEV11: !IODEV.12, U12.Y3
- new net !IODEV12: !IODEV.13, U12.Y4
- new net !IODEV13: !IODEV.14, U12.Y5
- new net !IODEV14: !IODEV.15, U12.Y6
- new net !IODEV15: !IODEV.16, U12.Y7
- new net !IODEV2: !IODEV.3, U11.Y2
- new net !IODEV3: !IODEV.4, U11.Y3
- new net !IODEV4: !IODEV.5, U11.Y4
- new net !IODEV5: !IODEV.6, U11.Y5
- new net !IODEV6: !IODEV.7, U11.Y6
- new net !IODEV7: !IODEV.8, U11.Y7
- new net !IODEV8: !IODEV.9, U12.Y0
- new net !IODEV9: !IODEV.10, U12.Y1
- new net !IO_SELECT_BANK0: U11.!G2B, U13.Y0
- new net !IO_SELECT_BANK1: U12.!G2A, U13.Y1
- new net !SCR0_CP: U16.1Y, U9.4A, U9.4B
- new net !SCR0_ROM_EN: U10.Q0, U6.1B, U9.3A, U9.3B
- new net N$1: U13.!G2B, U14.Y0
- new net N$2: U14.!G2B, U15.Y0
- new net N$3: U15.!G2B, U17.Y0
- new net SCR0_CP: U10.CP, U9.4Y
- net !IORQ: now also U11.!G2A, U12.!G2B, U13.!G2A, U14.!G2A, U15.!G2A, U17.!G2A
- net !M1: now also U11.G1, U12.G1, U13.G1, U14.G1, U15.G1, U17.G1
- net !RESET: now also U10.!MR
- net !WR: now also U16.1B
- net ADDR0: now also U11.A, U12.A
- net ADDR1: now also U11.B, U12.B
- net ADDR10: now also U15.B
- net ADDR11: now also U15.C
- net ADDR12: now also U17.A
- net ADDR13: now also U17.B
- net ADDR14: now also U17.C
- net ADDR15: now also U17.!G2B
- net ADDR2: now also U11.C, U12.C
- net ADDR3: now also U13.A
- net ADDR4: now also U13.B
- net ADDR5: now also U13.C
- net ADDR6: now also U14.A
- net ADDR7: now also U14.B
- net ADDR8: now also U14.C
- net ADDR9: now also U15.A
- net DATA0: now also U10.D0
- net DATA1: now also U10.D1
- net DATA2: now also U10.D2
- net DATA3: now also U10.D3
- net DATA4: now also U10.D4
- net DATA5: now also U10.D5
- net DATA6: now also U10.D6
- net DATA7: now also U10.D7
- net GND: now also !IODEV.1, P3.14, U10.GND, U11.GND, U12.GND, U13.GND, U14.GND, U15.GND, U16.GND, U17.GND
- net VCC: now also U10.VCC, U11.VCC, U12.VCC, U13.VCC, U14.VCC, U15.VCC, U16.VCC, U17.VCC
Other:
- note added: "IO Device Selector"
- note added: "SCR0 - System Control Register 0"
- moved on the sheet: C10, C11, C12, C13, C14, C15, C8, C9, P1, P2, P3, P4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
